File: Front-Control-Board/Front-Control-Board-Design/Front Board/USB-interface.kicad_sch (KiCad schematic)
At the start: 11 parts

Commit message: Front board finished schematic
Parts:
- C10, C9: renamed from C?; footprint (none) -> Capacitor_SMD:C_0603_1608Metric_Pad1.08x0.95mm_HandSolder
- R10, R11, R12, R13, R8, R9: renamed from R?; footprint (none) -> Resistor_SMD:R_0603_1608Metric_Pad0.98x0.95mm_HandSolder
- gave numbers to parts that had none: 3
Changed lines of the file:
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@@
     (stroke (width 0) (type default) (color 0 0 0 0))
   )
-  (wire (pts (xy 90.17 85.725) (xy 90.17 93.345))
+  (wire (pts (xy 90.17 85.725) (xy 90.17 93.726))
     (stroke (width 0) (type default) (color 0 0 0 0))
   )
@@
     (stroke (width 0) (type default) (color 0 0 0 0))
   )
-  (wire (pts (xy 90.17 93.345) (xy 93.98 93.345))
+  (wire (pts (xy 90.17 93.726) (xy 95.504 93.726))
     (stroke (width 0) (type default) (color 0 0 0 0))
   )
@@
     (effects (font (size 1.27 1.27)) (justify left bottom))
   )
-  (label "EN" (at 92.71 45.72 180)
-    (effects (font (size 1.27 1.27)) (justify right bottom))
-  )
   (label "DTR" (at 43.18 56.515 180)
-    (effects (font (size 1.27 1.27)) (justify right bottom))
-  )
-  (label "IO0" (at 93.98 93.345 180)
     (effects (font (size 1.27 1.27)) (justify right bottom))
   )
@@
     )
   )
+  (global_label "EN" (shape input) (at 92.71 45.72 0) (fields_autoplaced)
+    (effects (font (size 1.27 1.27)) (justify left))
+    (property "Intersheet References" "${INTERSHEET_REFS}" (id 0) (at 97.6026 45.6406 0)
+      (effects (font (size 1.27 1.27)) (justify left) hide)
+    )
+  )
+  (global_label "IO0" (shape input) (at 95.504 93.726 0) (fields_autoplaced)
+    (effects (font (size 1.27 1.27)) (justify left))
+    (property "Intersheet References" "${INTERSHEET_REFS}" (id 0) (at 101.0619 93.6466 0)
+      (effects (font (size 1.27 1.27)) (justify left) hide)
+    )
+  )
   (symbol (lib_id "Device:R") (at 165.608 74.676 90) (unit 1)
     (in_bom yes) (on_board yes)
-    (property "Reference" "R?" (id 0) (at 165.608 72.644 90))
+    (property "Reference" "R12" (id 0) (at 165.608 72.644 90))
     (property "Value" "10k" (id 1) (at 165.608 74.676 90))
-    (property "Footprint" "" (id 2) (at 165.608 76.454 90)
+    (property "Footprint" "Resistor_SMD:R_0603_1608Metric_Pad0.98x0.95mm_HandSolder" (id 2) (at 165.608 76.454 90)
       (effects (font (size 1.27 1.27)) hide)
     )
@@
   (symbol (lib_id "Transistor_BJT:S8050") (at 87.63 56.515 0) (unit 1)
     (in_bom yes) (on_board yes) (fields_autoplaced)
-    (property "Reference" "Q?" (id 0) (at 92.71 55.2449 0)
+    (property "Reference" "Q2" (id 0) (at 92.71 55.2449 0)
       (effects (font (size 1.27 1.27)) (justify left))
     )
@@
   (symbol (lib_id "Device:C") (at 149.098 28.194 90) (unit 1)
     (in_bom yes) (on_board yes)
-    (property "Reference" "C?" (id 0) (at 146.558 26.67 90))
+    (property "Reference" "C9" (id 0) (at 146.558 26.67 90))
     (property "Value" "4.7uF" (id 1) (at 149.098 31.496 90))
-    (property "Footprint" "" (id 2) (at 152.908 27.2288 0)
+    (property "Footprint" "Capacitor_SMD:C_0603_1608Metric_Pad1.08x0.95mm_HandSolder" (id 2) (at 152.908 27.2288 0)
       (effects (font (size 1.27 1.27)) hide)
     )
@@
   (symbol (lib_id "Device:C") (at 149.098 36.576 90) (unit 1)
     (in_bom yes) (on_board yes)
-    (property "Reference" "C?" (id 0) (at 146.05 35.306 90))
+    (property "Reference" "C10" (id 0) (at 146.05 35.306 90))
     (property "Value" "0.1uF" (id 1) (at 149.098 39.624 90))
-    (property "Footprint" "" (id 2) (at 152.908 35.6108 0)
+    (property "Footprint" "Capacitor_SMD:C_0603_1608Metric_Pad1.08x0.95mm_HandSolder" (id 2) (at 152.908 35.6108 0)
       (effects (font (size 1.27 1.27)) hide)
     )
@@
   (symbol (lib_id "power:GND") (at 117.602 74.422 0) (unit 1)
     (in_bom yes) (on_board yes) (fields_autoplaced)
-    (property "Reference" "#PWR?" (id 0) (at 117.602 80.772 0)
+    (property "Reference" "#PWR0122" (id 0) (at 117.602 80.772 0)
       (effects (font (size 1.27 1.27)) hide)
     )
@@
   (symbol (lib_id "Device:R") (at 63.5 56.515 90) (unit 1)
     (in_bom yes) (on_board yes)
-    (property "Reference" "R?" (id 0) (at 63.5 54.61 90))
+    (property "Reference" "R9" (id 0) (at 63.5 54.61 90))
     (property "Value" "10K" (id 1) (at 63.5 56.515 90))
-    (property "Footprint" "" (id 2) (at 63.5 58.293 90)
+    (property "Footprint" "Resistor_SMD:R_0603_1608Metric_Pad0.98x0.95mm_HandSolder" (id 2) (at 63.5 58.293 90)
       (effects (font (size 1.27 1.27)) hide)
     )
@@
   (symbol (lib_id "Device:R") (at 123.444 49.276 90) (unit 1)
     (in_bom yes) (on_board yes)
-    (property "Reference" "R?" (id 0) (at 123.444 47.244 90))
+    (property "Reference" "R8" (id 0) (at 123.444 47.244 90))
     (property "Value" "2k" (id 1) (at 123.444 49.276 90))
-    (property "Footprint" "" (id 2) (at 123.444 51.054 90)
+    (property "Footprint" "Resistor_SMD:R_0603_1608Metric_Pad0.98x0.95mm_HandSolder" (id 2) (at 123.444 51.054 90)
       (effects (font (size 1.27 1.27)) hide)
     )
@@
   (symbol (lib_id "Device:R") (at 113.792 61.976 90) (unit 1)
     (in_bom yes) (on_board yes)
-    (property "Reference" "R?" (id 0) (at 113.792 59.944 90))
+    (property "Reference" "R10" (id 0) (at 113.792 59.944 90))
     (property "Value" "22.1k" (id 1) (at 113.792 61.976 90))
-    (property "Footprint" "" (id 2) (at 113.792 63.754 90)
+    (property "Footprint" "Resistor_SMD:R_0603_1608Metric_Pad0.98x0.95mm_HandSolder" (id 2) (at 113.792 63.754 90)
       (effects (font (size 1.27 1.27)) hide)
     )
@@
   (symbol (lib_id "Device:R") (at 117.602 70.612 0) (unit 1)
     (in_bom yes) (on_board yes)
-    (property "Reference" "R?" (id 0) (at 119.38 69.3419 0)
+    (property "Reference" "R11" (id 0) (at 119.38 69.3419 0)
       (effects (font (size 1.27 1.27)) (justify left))
     )
@@
       (effects (font (size 1.27 1.27)) (justify left))
     )
-    (property "Footprint" "" (id 2) (at 115.824 70.612 90)
+    (property "Footprint" "Resistor_SMD:R_0603_1608Metric_Pad0.98x0.95mm_HandSolder" (id 2) (at 115.824 70.612 90)
       (effects (font (size 1.27 1.27)) hide)
     )
@@
   (symbol (lib_id "power:GND") (at 142.24 110.236 0) (unit 1)
     (in_bom yes) (on_board yes) (fields_autoplaced)
-    (property "Reference" "#PWR?" (id 0) (at 142.24 116.586 0)
+    (property "Reference" "#PWR0123" (id 0) (at 142.24 116.586 0)
       (effects (font (size 1.27 1.27)) hide)
     )
@@
   (symbol (lib_id "power:GND") (at 180.594 74.676 0) (unit 1)
     (in_bom yes) (on_board yes)
-    (property "Reference" "#PWR?" (id 0) (at 180.594 81.026 0)
+    (property "Reference" "#PWR0126" (id 0) (at 180.594 81.026 0)
       (effects (font (size 1.27 1.27)) hide)
     )
@@
   (symbol (lib_id "power:VDD") (at 142.24 23.114 0) (unit 1)
     (in_bom yes) (on_board yes) (fields_autoplaced)
-    (property "Reference" "#PWR?" (id 0) (at 142.24 26.924 0)
+    (property "Reference" "#PWR0124" (id 0) (at 142.24 26.924 0)
       (effects (font (size 1.27 1.27)) hide)
     )
@@
   (symbol (lib_id "Transistor_BJT:S8050") (at 87.63 80.645 0) (mirror x) (unit 1)
     (in_bom yes) (on_board yes) (fields_autoplaced)
-    (property "Reference" "Q?" (id 0) (at 92.71 79.3749 0)
+    (property "Reference" "Q3" (id 0) (at 92.71 79.3749 0)
       (effects (font (size 1.27 1.27)) (justify left))
     )
@@
   (symbol (lib_id "power:GND") (at 159.258 36.576 0) (unit 1)
     (in_bom yes) (on_board yes) (fields_autoplaced)
-    (property "Reference" "#PWR?" (id 0) (at 159.258 42.926 0)
+    (property "Reference" "#PWR0125" (id 0) (at 159.258 42.926 0)
       (effects (font (size 1.27 1.27)) hide)
     )
@@
   (symbol (lib_id "Device:R") (at 63.5 80.645 90) (unit 1)
     (in_bom yes) (on_board yes)
-    (property "Reference" "R?" (id 0) (at 63.5 78.74 90))
+    (property "Reference" "R13" (id 0) (at 63.5 78.74 90))
     (property "Value" "10K" (id 1) (at 63.5 80.645 90))
-    (property "Footprint" "" (id 2) (at 63.5 82.423 90)
+    (property "Footprint" "Resistor_SMD:R_0603_1608Metric_Pad0.98x0.95mm_HandSolder" (id 2) (at 63.5 82.423 90)
       (effects (font (size 1.27 1.27)) hide)
     )
@@
   (symbol (lib_id "Interface_USB:CP2102N-Axx-xQFN28") (at 142.24 77.216 0) (unit 1)
     (in_bom yes) (on_board yes) (fields_autoplaced)
-    (property "Reference" "U?" (id 0) (at 144.2594 110.871 0)
-      (effects (font (size 1.27 1.27)) (justify left))
-    )
+    (property "Reference" "U4" (id 0) (at 144.2594 110.871 0)
+      (effects (font (size 1.27 1.27)) (justify left))
+    )
