File: Wheel-Control-Board-Design/BoardV1Proto Backup/BoardV1Proto.kicad_sch (KiCad schematic)
At the start: 17 parts

Commit message: Re adding work from 11/11/2022
Un messing up by adding another version from before a push
Parts:
- removed D?: LED, symbol Device:LED
- removed R?: R, symbol Device:R
- removed SW?: SW_Push, symbol Switch:SW_Push
- added C?: 2.2µF, symbol Device:C
- added C?: .33µF, symbol Device:C
- added R?: (0~300k), symbol Device:R
Connections:
- net +3V3: now also U?.4 (VOUT), C?.1; no longer U?.2 (CHIP_PU)
- net Drive Mode Select: no longer U?.6 (VDET_2/GPIO35/ADC1_CH7)
- net GND: now also U?.3 (Gnd), C?.2, C?.2
- net LCD Mode Button: no longer U?.5 (VDET_1/GPIO34/ADC1_CH6)
- net VCC: now also U?.2 (VIN), C?.1, R?.1
- net at U?.1 (CONTROL): now also R?.2
- net Brake Regen: no longer names the net of U?.4 (SENSOR_VN/GPIO39/ADC1_CH3)
- net Brake Regen: no longer RV?.2
- net RTD Button: no longer names the net of U?.7 (32K_XP/GPIO32/ADC1_CH4)
- net RTD Button LED: no longer names the net of U?.8 (32K_XN/GPIO33/ADC1_CH5)
Other:
- note added: "LCD screen Connector"
- note added: "Power in to 3v3"
- moved on the sheet: BT?, J?, R?, RV?, SW?, U?
