File: Rear-Control-Board/rear-control-board-Design/FAULT_LATCHER.kicad_sch (KiCad schematic)
At the start: 11 parts, among them J4 JST-B2B-VERT-2PIN, J5 JST-B2B-VERT-2PIN, K2 G5V-2, K3 G5V-2

Commit message: pcb Done? check SD
Parts:
- gave numbers to parts that had none: 2
Connections:
- net +3V3 renamed VDD
Changed lines of the file:
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@@
     (pin "1")
   )
-  (symbol (lib_id "power:+3.3V") (at 43.18 72.39 0) (unit 1)
-    (in_bom yes) (on_board yes)
-    (property "Reference" "#PWR0120" (id 0) (at 43.18 76.2 0)
+  (symbol (lib_id "power:VDD") (at 43.18 72.39 0) (unit 1)
+    (in_bom yes) (on_board yes) (fields_autoplaced)
+    (property "Reference" "#PWR0110" (id 0) (at 43.18 76.2 0)
       (effects (font (size 1.27 1.27)) hide)
     )
-    (property "Value" "+3.3V" (id 1) (at 43.561 67.9958 0))
+    (property "Value" "VDD" (id 1) (at 43.18 66.802 0))
     (property "Footprint" "" (id 2) (at 43.18 72.39 0)
       (effects (font (size 1.27 1.27)) hide)
@@
     (pin "1")
   )
-  (symbol (lib_id "power:+3.3V") (at 74.295 166.37 180) (unit 1)
-    (in_bom yes) (on_board yes) (fields_autoplaced)
-    (property "Reference" "#PWR?" (id 0) (at 74.295 162.56 0)
-      (effects (font (size 1.27 1.27)) hide)
-    )
-    (property "Value" "+3.3V" (id 1) (at 74.295 171.45 0))
-    (property "Footprint" "" (id 2) (at 74.295 166.37 0)
-      (effects (font (size 1.27 1.27)) hide)
-    )
-    (property "Datasheet" "" (id 3) (at 74.295 166.37 0)
-      (effects (font (size 1.27 1.27)) hide)
-    )
-    (pin "1")
-  )
   (symbol (lib_id "Transistor_BJT:FFB5551") (at 71.755 151.765 0) (unit 1)
     (in_bom yes) (on_board yes) (fields_autoplaced)
-    (property "Reference" "Q?" (id 0) (at 77.47 150.4949 0)
+    (property "Reference" "Q1" (id 0) (at 77.47 150.4949 0)
       (effects (font (size 1.27 1.27)) (justify left))
     )
@@
   (symbol (lib_id "power:GND") (at 95.25 143.51 0) (unit 1)
     (in_bom yes) (on_board yes) (fields_autoplaced)
-    (property "Reference" "#PWR?" (id 0) (at 95.25 149.86 0)
+    (property "Reference" "#PWR0109" (id 0) (at 95.25 149.86 0)
       (effects (font (size 1.27 1.27)) hide)
     )
@@
   (symbol (lib_id "Device:R") (at 95.25 139.7 0) (unit 1)
     (in_bom yes) (on_board yes)
-    (property "Reference" "R?" (id 0) (at 97.79 138.4299 0)
+    (property "Reference" "R10" (id 0) (at 97.79 138.4299 0)
       (effects (font (size 1.27 1.27)) (justify left))
     )
@@
     (pin "2")
   )
+  (symbol (lib_id "power:VDD") (at 74.295 166.37 90) (unit 1)
+    (in_bom yes) (on_board yes) (fields_autoplaced)
+    (property "Reference" "#PWR0120" (id 0) (at 78.105 166.37 0)
+      (effects (font (size 1.27 1.27)) hide)
+    )
+    (property "Value" "VDD" (id 1) (at 75.311 166.3699 90)
+      (effects (font (size 1.27 1.27)) (justify right))
+    )
+    (property "Footprint" "" (id 2) (at 74.295 166.37 0)
+      (effects (font (size 1.27 1.27)) hide)
+    )
+    (property "Datasheet" "" (id 3) (at 74.295 166.37 0)
+      (effects (font (size 1.27 1.27)) hide)
+    )
+    (pin "1")
+  )
 )

Commit message: rcb
Parts:
- R10: footprint (none) -> Resistor_SMD:R_0603_1608Metric_Pad0.98x0.95mm_HandSolder
Changed lines of the file:
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@@
       (effects (font (size 1.27 1.27)) (justify left))
     )
-    (property "Footprint" "" (id 2) (at 93.472 139.7 90)
+    (property "Footprint" "Resistor_SMD:R_0603_1608Metric_Pad0.98x0.95mm_HandSolder" (id 2) (at 93.472 139.7 90)
       (effects (font (size 1.27 1.27)) hide)
     )

Commit message: update
Parts:
- removed Q1: B5584, Package_TO_SOT_SMD:SOT-363_SC-70-6, symbol Transistor_BJT:FFB5551
- removed R10: 470, Resistor_SMD:R_0603_1608Metric_Pad0.98x0.95mm_HandSolder, symbol Device:R
Changed lines of the file:
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@@
   (junction (at 145.415 99.695) (diameter 0) (color 0 0 0 0)
-  )
-  (junction (at 95.25 135.89) (diameter 0) (color 0 0 0 0)
   )
   (junction (at 135.255 67.31) (diameter 0) (color 0 0 0 0)
@@
   (no_connect (at 137.16 59.69))
   (no_connect (at 137.16 49.53))
-  (wire (pts (xy 63.5 151.765) (xy 66.675 151.765))
-    (stroke (width 0) (type default) (color 0 0 0 0))
-  )
   (wire (pts (xy 155.575 84.455) (xy 155.575 67.31))
     (stroke (width 0) (type default) (color 0 0 0 0))
@@
     (stroke (width 0) (type default) (color 0 0 0 0))
   )
-  (bus (pts (xy 119.38 122.555) (xy 119.38 175.26))
-    (stroke (width 0) (type default) (color 0 0 0 0))
-  )
   (wire (pts (xy 97.79 65.405) (xy 97.79 67.31))
     (stroke (width 0) (type default) (color 0 0 0 0))
@@
     (stroke (width 0) (type default) (color 0 0 0 0))
   )
-  (wire (pts (xy 74.295 156.845) (xy 74.295 166.37))
-    (stroke (width 0) (type default) (color 0 0 0 0))
-  )
-  (wire (pts (xy 74.295 135.89) (xy 95.25 135.89))
-    (stroke (width 0) (type default) (color 0 0 0 0))
-  )
-  (wire (pts (xy 95.25 135.89) (xy 106.68 135.89))
-    (stroke (width 0) (type default) (color 0 0 0 0))
-  )
   (wire (pts (xy 135.255 54.61) (xy 135.255 67.31))
     (stroke (width 0) (type default) (color 0 0 0 0))
@@
     (stroke (width 0) (type default) (color 0 0 0 0))
   )
-  (bus (pts (xy 46.99 122.555) (xy 46.99 175.26))
-    (stroke (width 0) (type default) (color 0 0 0 0))
-  )
   (wire (pts (xy 155.575 84.455) (xy 155.575 99.695))
     (stroke (width 0) (type default) (color 0 0 0 0))
@@
     (stroke (width 0) (type default) (color 0 0 0 0))
   )
-  (bus (pts (xy 46.99 122.555) (xy 119.38 122.555))
-    (stroke (width 0) (type default) (color 0 0 0 0))
-  )
   (wire (pts (xy 135.255 67.31) (xy 137.16 67.31))
     (stroke (width 0) (type default) (color 0 0 0 0))
@@
     (stroke (width 0) (type default) (color 0 0 0 0))
   )
-  (bus (pts (xy 119.38 175.26) (xy 46.99 175.26))
-    (stroke (width 0) (type default) (color 0 0 0 0))
-  )
   (wire (pts (xy 60.96 80.01) (xy 60.96 67.31))
     (stroke (width 0) (type default) (color 0 0 0 0))
@@
   )
   (wire (pts (xy 145.415 99.695) (xy 155.575 99.695))
-    (stroke (width 0) (type default) (color 0 0 0 0))
-  )
-  (wire (pts (xy 74.295 146.685) (xy 74.295 135.89))
     (stroke (width 0) (type default) (color 0 0 0 0))
   )
@@
   (label "IMD_SWITCH" (at 135.255 67.31 180)
     (effects (font (size 1.27 1.27)) (justify right bottom))
-  )
-  (label "BMS_IND" (at 106.68 135.89 0)
-    (effects (font (size 1.27 1.27) bold italic) (justify left bottom))
   )
   (global_label "INT_12V" (shape input) (at 97.79 65.405 0) (fields_autoplaced)
@@
     (property "Intersheet References" "${INTERSHEET_REFS}" (id 0) (at 107.4923 65.3256 0)
       (effects (font (size 1.27 1.27)) (justify left) hide)
-    )
-  )
-  (global_label "BMS_SW" (shape input) (at 63.5 151.765 180) (fields_autoplaced)
-    (effects (font (size 1.27 1.27) bold italic) (justify right))
-    (property "Intersheet References" "${INTERSHEET_REFS}" (id 0) (at 53.1703 151.638 0)
-      (effects (font (size 1.27 1.27) bold italic) (justify right) hide)
     )
   )
@@
     (pin "1")
   )
-  (symbol (lib_id "Transistor_BJT:FFB5551") (at 71.755 151.765 0) (unit 1)
-    (in_bom yes) (on_board yes) (fields_autoplaced)
-    (property "Reference" "Q1" (id 0) (at 77.47 150.4949 0)
-      (effects (font (size 1.27 1.27)) (justify left))
-    )
-    (property "Value" "B5584" (id 1) (at 77.47 153.0349 0)
-      (effects (font (size 1.27 1.27)) (justify left))
-    )
-    (property "Footprint" "Package_TO_SOT_SMD:SOT-363_SC-70-6" (id 2) (at 76.835 149.225 0)
-      (effects (font (size 1.27 1.27)) hide)
-    )
-    (property "Datasheet" "https://www.onsemi.com/pub/Collateral/FFB5551-D.PDF" (id 3) (at 71.755 151.765 0)
-      (effects (font (size 1.27 1.27)) hide)
-    )
-    (pin "1")
-    (pin "2")
-    (pin "6")
-  )
-  (symbol (lib_id "power:GND") (at 95.25 143.51 0) (unit 1)
-    (in_bom yes) (on_board yes) (fields_autoplaced)
-    (property "Reference" "#PWR0109" (id 0) (at 95.25 149.86 0)
-      (effects (font (size 1.27 1.27)) hide)
-    )
-    (property "Value" "GND" (id 1) (at 95.25 148.59 0))
-    (property "Footprint" "" (id 2) (at 95.25 143.51 0)
-      (effects (font (size 1.27 1.27)) hide)
-    )
-    (property "Datasheet" "" (id 3) (at 95.25 143.51 0)
-      (effects (font (size 1.27 1.27)) hide)
-    )
-    (pin "1")
-  )
   (symbol (lib_id "Device:R") (at 135.255 95.885 0) (unit 1)
     (in_bom yes) (on_board yes)
@@
     (pin "2")
   )
-  (symbol (lib_id "Device:R") (at 95.25 139.7 0) (unit 1)
-    (in_bom yes) (on_board yes)
-    (property "Reference" "R10" (id 0) (at 97.79 138.4299 0)
-      (effects (font (size 1.27 1.27)) (justify left))
-    )
-    (property "Value" "470" (id 1) (at 95.25 141.605 90)
-      (effects (font (size 1.27 1.27)) (justify left))
-    )
-    (property "Footprint" "Resistor_SMD:R_0603_1608Metric_Pad0.98x0.95mm_HandSolder" (id 2) (at 93.472 139.7 90)
-      (effects (font (size 1.27 1.27)) hide)
-    )
-    (property "Datasheet" "~" (id 3) (at 95.25 139.7 0)
-      (effects (font (size 1.27 1.27)) hide)
-    )
-    (pin "1")
-    (pin "2")
-  )
-  (symbol (lib_id "power:VDD") (at 74.295 166.37 90) (unit 1)
-    (in_bom yes) (on_board yes) (fields_autoplaced)
-    (property "Reference" "#PWR0120" (id 0) (at 78.105 166.37 0)
-      (effects (font (size 1.27 1.27)) hide)
-    )
-    (property "Value" "VDD" (id 1) (at 75.311 166.3699 90)
-      (effects (font (size 1.27 1.27)) (justify right))
-    )
-    (property "Footprint" "" (id 2) (at 74.295 166.37 0)
-      (effects (font (size 1.27 1.27)) hide)
-    )
-    (property "Datasheet" "" (id 3) (at 74.295 166.37 0)
-      (effects (font (size 1.27 1.27)) hide)
-    )
-    (pin "1")
-  )
 )
