File: Rear-Control-Board/rear-control-board-Design/FET_OUTPUT.kicad_sch (KiCad schematic)
At the start: 16 parts, among them U5 BV1HAL45EFJ, U6 BV1HAL45EFJ, U7 BV1HAL45EFJ

Commit message: update
Parts:
- added Q?: PSMN5R2-60YL, Package_TO_SOT_SMD:LFPAK56, symbol Transistor_FET:PSMN5R2-60YL
- added R?: R, symbol Device:R
Connections:
- net GND: now also Q?.1 (S), Q?.2 (S), Q?.3 (S)
- net PUMP_CTRL: now also R?.1
- net PUMP_OUT: now also Q?.5 (D)
- new net: Q?.4 (G), R?.2
Other:
- note added: "Replace load switch with"
Changed lines of the file:
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@@
+    (stroke (width 0) (type default) (color 0 0 0 0))
+  )
+  (wire (pts (xy 144.018 121.793) (xy 149.733 121.793))
     (stroke (width 0) (type default) (color 0 0 0 0))
   )
@@
     (stroke (width 0) (type default) (color 0 0 0 0))
   )
+  (wire (pts (xy 170.053 113.665) (xy 170.053 116.713))
+    (stroke (width 0) (type default) (color 0 0 0 0))
+  )
   (wire (pts (xy 121.285 78.105) (xy 121.285 79.375))
+    (stroke (width 0) (type default) (color 0 0 0 0))
+  )
+  (wire (pts (xy 157.353 121.793) (xy 162.433 121.793))
     (stroke (width 0) (type default) (color 0 0 0 0))
   )
@@
     (effects (font (size 1.27 1.27) bold italic) (justify left bottom))
   )
+  (text "Replace load switch with" (at 175.768 127.381 0)
+    (effects (font (size 1.27 1.27)) (justify left bottom))
+  )
   (text "2.2mA current \nlimiting resistor " (at 45.974 60.96 0)
     (effects (font (size 1.27 1.27)) (justify left bottom))
@@
     (effects (font (size 1.27 1.27)) (justify right))
   )
+  (hierarchical_label "PUMP_12V" (shape input) (at 170.053 109.982 180)
+    (effects (font (size 1.27 1.27)) (justify right))
+  )
   (hierarchical_label "Brake_out" (shape input) (at 204.47 82.55 180)
     (effects (font (size 1.27 1.27) bold italic) (justify right))
@@
     (effects (font (size 1.27 1.27)) (justify right))
   )
+  (hierarchical_label "PUMP_OUT" (shape input) (at 170.053 113.665 0)
+    (effects (font (size 1.27 1.27)) (justify left))
+  )
   (hierarchical_label "BRAKE_OUT" (shape input) (at 178.435 78.74 0)
     (effects (font (size 1.27 1.27)) (justify left))
@@
     (effects (font (size 1.27 1.27)) (justify right))
   )
+  (hierarchical_label "PUMP_CTRL" (shape input) (at 144.018 121.793 180)
+    (effects (font (size 1.27 1.27)) (justify right))
+  )
   (hierarchical_label "BRAKE_CTRL" (shape input) (at 151.765 82.55 180)
     (effects (font (size 1.27 1.27)) (justify right))
@@
   (hierarchical_label "BRAKE_12V" (shape input) (at 189.23 62.23 180)
     (effects (font (size 1.27 1.27)) (justify right))
+  )
+  (symbol (lib_id "power:GND") (at 170.053 126.873 0) (unit 1)
+    (in_bom yes) (on_board yes) (fields_autoplaced)
+    (property "Reference" "#PWR?" (id 0) (at 170.053 133.223 0)
+      (effects (font (size 1.27 1.27)) hide)
+    )
+    (property "Value" "GND" (id 1) (at 170.053 132.08 0))
+    (property "Footprint" "" (id 2) (at 170.053 126.873 0)
+      (effects (font (size 1.27 1.27)) hide)
+    )
+    (property "Datasheet" "" (id 3) (at 170.053 126.873 0)
+      (effects (font (size 1.27 1.27)) hide)
+    )
+    (pin "1")
   )
   (symbol (lib_id "power:GND") (at 220.345 82.55 0) (unit 1)
@@
     (pin "1")
   )
+  (symbol (lib_id "Device:R") (at 153.543 121.793 90) (unit 1)
+    (in_bom yes) (on_board yes) (fields_autoplaced)
+    (property "Reference" "R?" (id 0) (at 153.543 115.697 90))
+    (property "Value" "R" (id 1) (at 153.543 118.237 90))
+    (property "Footprint" "" (id 2) (at 153.543 123.571 90)
+      (effects (font (size 1.27 1.27)) hide)
+    )
+    (property "Datasheet" "~" (id 3) (at 153.543 121.793 0)
+      (effects (font (size 1.27 1.27)) hide)
+    )
+    (pin "1")
+    (pin "2")
+  )
+  (symbol (lib_id "Transistor_FET:PSMN5R2-60YL") (at 167.513 121.793 0) (unit 1)
+    (in_bom yes) (on_board yes) (fields_autoplaced)
+    (property "Reference" "Q?" (id 0) (at 172.72 120.5229 0)
+      (effects (font (size 1.27 1.27)) (justify left))
+    )
+    (property "Value" "PSMN5R2-60YL" (id 1) (at 172.72 123.0629 0)
+      (effects (font (size 1.27 1.27)) (justify left))
+    )
+    (property "Footprint" "Package_TO_SOT_SMD:LFPAK56" (id 2) (at 171.323 121.793 0)
+      (effects (font (size 1.27 1.27)) hide)
+    )
+    (property "Datasheet" "https://assets.nexperia.com/documents/data-sheet/PSMN5R2-60YL.pdf" (id 3) (at 167.513 121.793 0)
+      (effects (font (size 1.27 1.27)) hide)
+    )
+    (pin "1")
+    (pin "2")
+    (pin "3")
+    (pin "4")
+    (pin "5")
+  )
   (symbol (lib_id "power:GND") (at 132.08 69.85 0) (unit 1)

Commit message: pcb Done? check SD
Parts:
- removed Q?: PSMN5R2-60YL, Package_TO_SOT_SMD:LFPAK56, symbol Transistor_FET:PSMN5R2-60YL
- removed R1, R14, R16: 20k, Resistor_SMD:R_0603_1608Metric_Pad0.98x0.95mm_HandSolder, symbol Device:R
- removed R15, R9: 50k, Resistor_SMD:R_0603_1608Metric_Pad0.98x0.95mm_HandSolder, symbol Device:R
- removed R17: 200k, Resistor_SMD:R_0603_1608Metric_Pad0.98x0.95mm_HandSolder, symbol Device:R
- removed R?: 10k, symbol Device:R
- removed R?: R, symbol Device:R
- removed U5, U6, U7: BV1HAL45EFJ, Package_SO:HTSOP-8-1EP_3.9x4.9mm_P1.27mm_EP2.4x3.2mm_ThermalVias, symbol AERO_Symbols:BV1HAL45EFJ
- added Q3, Q4, Q?: PSMN5R2-60YL, Package_TO_SOT_SMD:LFPAK56, symbol Transistor_FET:PSMN5R2-60YL
Connections:
- net BRAKE_12V: now also Q?.5 (D)
- net FAN_12V: now also Q4.5 (D)
- net GND: now also Q3.1 (S), Q3.2 (S), Q3.3 (S), Q4.1 (S), Q4.2 (S), Q4.3 (S), Q?.1 (S), Q?.2 (S), Q?.3 (S)
- net PUMP_12V: now also Q3.5 (D)
- net at R13.2: now also Q?.4 (G)
- net at R12.2: now also Q3.4 (G)
- net at R11.2: now also Q4.4 (G)
Other:
- note removed: "*On startup, all 0v, then signal high, out is 12v, signal low, out is 8.44v"
- note removed: "2.2mA current limiting resistor"
- note removed: "All three only go down to 8.5v when signal is low"
- note removed: "Change TO diffrent type of load switch"
- note removed: "From STM32 3.3 High 0v low"
- note removed: "NOTE: Pump is always on and does not need switching was removed and is now always on. Brake works fine and is in place. Fan was to high of a current draw for the BV1HAL45EFJ so is currently always on, in the future will find an apropriate load switch."
- note removed: "Pulled to ground"
- note removed: "Replace load switch with"
- note removed: "Should be 50k"
- note removed: "Should limit between 50-100uA"
- moved on the sheet: C13, C3, R11, R12, R13

Commit message: rcb
Parts:
- gave numbers to parts that had none: 1
Changed lines of the file:
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@@
   (symbol (lib_id "Transistor_FET:PSMN5R2-60YL") (at 166.878 80.645 0) (unit 1)
     (in_bom yes) (on_board yes) (fields_autoplaced)
-    (property "Reference" "Q?" (id 0) (at 172.085 79.3749 0)
+    (property "Reference" "Q2" (id 0) (at 172.085 79.3749 0)
       (effects (font (size 1.27 1.27)) (justify left))
     )

Commit message: update
Parts:
- removed R11, R12, R13: 1.5K, Resistor_SMD:R_0603_1608Metric_Pad0.98x0.95mm_HandSolder, symbol Device:R
Connections:
- net BRAKE_CTRL: now also Q2.4 (G)
- net FAN_CTRL: now also Q4.4 (G)
- net PUMP_CTRL: now also Q3.4 (G)
Changed lines of the file:
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@@
 (kicad_sch (version 20211123) (generator eeschema)
   (paper "A4")
-  (wire (pts (xy 102.743 79.629) (xy 105.918 79.629))
+  (wire (pts (xy 95.123 79.629) (xy 105.918 79.629))
+    (stroke (width 0) (type default) (color 0 0 0 0))
+  )
+  (wire (pts (xy 154.178 80.645) (xy 161.798 80.645))
     (stroke (width 0) (type default) (color 0 0 0 0))
   )
@@
   )
   (wire (pts (xy 169.418 88.138) (xy 169.418 85.725))
+    (stroke (width 0) (type default) (color 0 0 0 0))
+  )
+  (wire (pts (xy 41.402 78.486) (xy 49.022 78.486))
     (stroke (width 0) (type default) (color 0 0 0 0))
   )
@@
     (pin "2")
   )
-  (symbol (lib_id "Device:R") (at 157.988 80.645 90) (unit 1)
-    (in_bom yes) (on_board yes)
-    (property "Reference" "R13" (id 0) (at 157.988 83.185 90))
-    (property "Value" "1.5K" (id 1) (at 157.988 80.645 90))
-    (property "Footprint" "Resistor_SMD:R_0603_1608Metric_Pad0.98x0.95mm_HandSolder" (id 2) (at 157.988 82.423 90)
-      (effects (font (size 1.27 1.27)) hide)
-    )
-    (property "Datasheet" "~" (id 3) (at 157.988 80.645 0)
-      (effects (font (size 1.27 1.27)) hide)
-    )
-    (pin "1")
-    (pin "2")
-  )
   (symbol (lib_id "Transistor_FET:PSMN5R2-60YL") (at 110.998 79.629 0) (unit 1)
     (in_bom yes) (on_board yes) (fields_autoplaced)
@@
     (pin "1")
   )
-  (symbol (lib_id "Device:R") (at 98.933 79.629 90) (unit 1)
-    (in_bom yes) (on_board yes)
-    (property "Reference" "R12" (id 0) (at 98.933 82.169 90))
-    (property "Value" "1.5K" (id 1) (at 98.933 79.629 90))
-    (property "Footprint" "Resistor_SMD:R_0603_1608Metric_Pad0.98x0.95mm_HandSolder" (id 2) (at 98.933 81.407 90)
-      (effects (font (size 1.27 1.27)) hide)
-    )
-    (property "Datasheet" "~" (id 3) (at 98.933 79.629 0)
-      (effects (font (size 1.27 1.27)) hide)
-    )
-    (pin "1")
-    (pin "2")
-  )
-  (symbol (lib_id "Device:R") (at 45.212 78.486 90) (unit 1)
-    (in_bom yes) (on_board yes)
-    (property "Reference" "R11" (id 0) (at 45.212 81.026 90))
-    (property "Value" "1.5K" (id 1) (at 45.212 78.486 90))
-    (property "Footprint" "Resistor_SMD:R_0603_1608Metric_Pad0.98x0.95mm_HandSolder" (id 2) (at 45.212 80.264 90)
-      (effects (font (size 1.27 1.27)) hide)
-    )
-    (property "Datasheet" "~" (id 3) (at 45.212 78.486 0)
-      (effects (font (size 1.27 1.27)) hide)
-    )
-    (pin "1")
-    (pin "2")
-  )
   (symbol (lib_id "Device:C") (at 181.356 68.834 0) (unit 1)
