File: Rear-Control-Board/rear-control-board-Design/Controller.kicad_sch (KiCad schematic)
At the start: 11 parts, among them U4 MAX33054EASA+T

Commit message: pcb Done? check SD
Parts:
- added J7: Micro_SD_Card, Connector_Card:microSD_HC_Wuerth_693072010801, symbol Connector:Micro_SD_Card
- gave numbers to parts that had none: 4
Connections:
- net GND: now also J7.6 (VSS), J7.9 (SHIELD)
- net SD_CS: now also J7.2 (DAT3/CD)
- net SD_MISO: now also J7.7 (DAT0)
- net SD_MOSI: now also J7.3 (CMD)
- net SD_SCK: now also J7.5 (CLK)
- net VDD: now also J7.4 (VDD)
- no-connect marks 0 -> 2
Changed lines of the file:
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@@
   (junction (at 248.92 136.525) (diameter 0) (color 0 0 0 0)
   )
+  (no_connect (at 101.346 152.527))
+  (no_connect (at 101.346 134.747))
   (wire (pts (xy 61.849 56.642) (xy 84.582 56.642))
     (stroke (width 0) (type default) (color 0 0 0 0))
@@
     (effects (font (size 1.27 1.27)) (justify left bottom))
   )
+  (label "SD_CS" (at 101.346 149.987 0)
+    (effects (font (size 1.27 1.27)) (justify left bottom))
+  )
   (label "CAN_MISO" (at 243.205 136.525 180)
     (effects (font (size 1.27 1.27)) (justify right bottom))
@@
     (effects (font (size 1.27 1.27)) (justify right bottom))
   )
+  (label "SD_SCK" (at 101.346 142.367 0)
+    (effects (font (size 1.27 1.27)) (justify left bottom))
+  )
   (label "SD_MISO" (at 84.582 69.342 180)
     (effects (font (size 1.27 1.27)) (justify right bottom))
   )
+  (label "SD_MOSI" (at 101.346 147.447 0)
+    (effects (font (size 1.27 1.27)) (justify left bottom))
+  )
   (label "CAN_MOSI" (at 154.432 41.402 0)
     (effects (font (size 1.27 1.27)) (justify left bottom))
@@
   )
   (label "TEMP_WATER_OUT" (at 154.432 71.882 0)
+    (effects (font (size 1.27 1.27)) (justify left bottom))
+  )
+  (label "SD_MISO" (at 101.346 137.287 0)
     (effects (font (size 1.27 1.27)) (justify left bottom))
   )
@@
   (symbol (lib_id "power:VDD") (at 265.684 77.216 0) (unit 1)
     (in_bom yes) (on_board yes) (fields_autoplaced)
-    (property "Reference" "#PWR?" (id 0) (at 265.684 81.026 0)
+    (property "Reference" "#PWR0128" (id 0) (at 265.684 81.026 0)
       (effects (font (size 1.27 1.27)) hide)
     )
@@
   (symbol (lib_id "power:GND") (at 31.369 57.15 0) (mirror y) (unit 1)
     (in_bom yes) (on_board yes)
-    (property "Reference" "#PWR?" (id 0) (at 31.369 63.5 0)
+    (property "Reference" "#PWR0133" (id 0) (at 31.369 63.5 0)
       (effects (font (size 1.27 1.27)) hide)
     )
@@
   (symbol (lib_id "power:GND") (at 84.582 71.882 270) (unit 1)
     (in_bom yes) (on_board yes)
-    (property "Reference" "#PWR?" (id 0) (at 78.232 71.882 0)
+    (property "Reference" "#PWR0123" (id 0) (at 78.232 71.882 0)
       (effects (font (size 1.27 1.27)) hide)
     )
@@
   (symbol (lib_id "power:GND") (at 45.339 61.595 0) (mirror y) (unit 1)
     (in_bom yes) (on_board yes)
-    (property "Reference" "#PWR?" (id 0) (at 45.339 67.945 0)
+    (property "Reference" "#PWR0132" (id 0) (at 45.339 67.945 0)
       (effects (font (size 1.27 1.27)) hide)
     )
@@
     (pin "1")
   )
+  (symbol (lib_id "power:VDD") (at 101.346 144.907 270) (unit 1)
+    (in_bom yes) (on_board yes) (fields_autoplaced)
+    (property "Reference" "#PWR0142" (id 0) (at 97.536 144.907 0)
+      (effects (font (size 1.27 1.27)) hide)
+    )
+    (property "Value" "VDD" (id 1) (at 105.41 144.9069 90)
+      (effects (font (size 1.27 1.27)) (justify left))
+    )
+    (property "Footprint" "" (id 2) (at 101.346 144.907 0)
+      (effects (font (size 1.27 1.27)) hide)
+    )
+    (property "Datasheet" "" (id 3) (at 101.346 144.907 0)
+      (effects (font (size 1.27 1.27)) hide)
+    )
+    (pin "1")
+  )
   (symbol (lib_id "power:GND") (at 226.314 94.361 0) (mirror y) (unit 1)
     (in_bom yes) (on_board yes) (fields_autoplaced)
@@
   (symbol (lib_id "Power_Protection:SP0502BAHT") (at 45.339 56.515 0) (mirror y) (unit 1)
     (in_bom yes) (on_board yes)
-    (property "Reference" "D?" (id 0) (at 46.863 56.261 0)
+    (property "Reference" "D6" (id 0) (at 46.863 56.261 0)
       (effects (font (size 1.27 1.27)) (justify left))
     )
@@
   (symbol (lib_id "power:GND") (at 154.432 38.862 90) (unit 1)
     (in_bom yes) (on_board yes) (fields_autoplaced)
-    (property "Reference" "#PWR?" (id 0) (at 160.782 38.862 0)
+    (property "Reference" "#PWR0114" (id 0) (at 160.782 38.862 0)
       (effects (font (size 1.27 1.27)) hide)
     )
@@
   (symbol (lib_id "power:GND") (at 59.309 68.707 0) (unit 1)
     (in_bom yes) (on_board yes)
-    (property "Reference" "#PWR?" (id 0) (at 59.309 75.057 0)
+    (property "Reference" "#PWR0134" (id 0) (at 59.309 75.057 0)
       (effects (font (size 1.27 1.27)) hide)
     )
@@
   (symbol (lib_id "power:VDD") (at 237.49 119.38 0) (unit 1)
     (in_bom yes) (on_board yes) (fields_autoplaced)
-    (property "Reference" "#PWR?" (id 0) (at 237.49 123.19 0)
+    (property "Reference" "#PWR0127" (id 0) (at 237.49 123.19 0)
       (effects (font (size 1.27 1.27)) hide)
     )
@@
     (pin "1")
   )
+  (symbol (lib_id "power:GND") (at 58.166 129.667 270) (unit 1)
+    (in_bom yes) (on_board yes) (fields_autoplaced)
+    (property "Reference" "#PWR0144" (id 0) (at 51.816 129.667 0)
+      (effects (font (size 1.27 1.27)) hide)
+    )
+    (property "Value" "GND" (id 1) (at 54.61 129.6669 90)
+      (effects (font (size 1.27 1.27)) (justify right))
+    )
+    (property "Footprint" "" (id 2) (at 58.166 129.667 0)
+      (effects (font (size 1.27 1.27)) hide)
+    )
+    (property "Datasheet" "" (id 3) (at 58.166 129.667 0)
+      (effects (font (size 1.27 1.27)) hide)
+    )
+    (pin "1")
+  )
   (symbol (lib_id "Power_Protection:SP0502BAHT") (at 59.309 63.627 0) (mirror y) (unit 1)
     (in_bom yes) (on_board yes)
-    (property "Reference" "D?" (id 0) (at 60.452 63.5 0)
+    (property "Reference" "D7" (id 0) (at 60.452 63.5 0)
       (effects (font (size 1.27 1.27)) (justify left))
     )
@@
   (symbol (lib_id "power:VDD") (at 243.84 119.38 0) (unit 1)
     (in_bom yes) (on_board yes) (fields_autoplaced)
-    (property "Reference" "#PWR?" (id 0) (at 243.84 123.19 0)
+    (property "Reference" "#PWR0126" (id 0) (at 243.84 123.19 0)
       (effects (font (size 1.27 1.27)) hide)
     )
@@
     (pin "1")
   )
+  (symbol (lib_id "Connector:Micro_SD_Card") (at 78.486 144.907 180) (unit 1)
+    (in_bom yes) (on_board yes) (fields_autoplaced)
+    (property "Reference" "J7" (id 0) (at 77.851 123.19 0))
+    (property "Value" "Micro_SD_Card" (id 1) (at 77.851 125.73 0))
+    (property "Footprint" "Connector_Card:microSD_HC_Wuerth_693072010801" (id 2) (at 49.276 152.527 0)
+      (effects (font (size 1.27 1.27)) hide)
+    )
+    (property "Datasheet" "http://katalog.we-online.de/em/datasheet/693072010801.pdf" (id 3) (at 78.486 144.907 0)
+      (effects (font (size 1.27 1.27)) hide)
+    )
+    (pin "1")
+    (pin "2")
+    (pin "3")
+    (pin "4")
+    (pin "5")
+    (pin "6")
+    (pin "7")
+    (pin "8")
+    (pin "9")
+  )
   (symbol (lib_id "power:VDD") (at 198.12 128.905 0) (unit 1)
     (in_bom yes) (on_board yes) (fields_autoplaced)
-    (property "Reference" "#PWR?" (id 0) (at 198.12 132.715 0)
+    (property "Reference" "#PWR0125" (id 0) (at 198.12 132.715 0)
       (effects (font (size 1.27 1.27)) hide)
     )
@@
   (symbol (lib_id "power:GND") (at 154.432 54.102 90) (unit 1)
     (in_bom yes) (on_board yes) (fields_autoplaced)
-    (property "Reference" "#PWR?" (id 0) (at 160.782 54.102 0)
+    (property "Reference" "#PWR0111" (id 0) (at 160.782 54.102 0)
       (effects (font (size 1.27 1.27)) hide)
     )
@@
   (symbol (lib_id "power:VDD") (at 227.584 76.581 0) (unit 1)
     (in_bom yes) (on_board yes) (fields_autoplaced)
-    (property "Reference" "#PWR?" (id 0) (at 227.584 80.391 0)
+    (property "Reference" "#PWR0131" (id 0) (at 227.584 80.391 0)
       (effects (font (size 1.27 1.27)) hide)
     )
@@
   (symbol (lib_id "power:VDD") (at 84.582 38.862 0) (unit 1)
     (in_bom yes) (on_board yes) (fields_autoplaced)
-    (property "Reference" "#PWR?" (id 0) (at 84.582 42.672 0)
+    (property "Reference" "#PWR0122" (id 0) (at 84.582 42.672 0)
       (effects (font (size 1.27 1.27)) hide)
     )
@@
     (pin "1")
   )
+  (symbol (lib_id "power:GND") (at 101.346 139.827 90) (unit 1)
+    (in_bom yes) (on_board yes) (fields_autoplaced)
+    (property "Reference" "#PWR0154" (id 0) (at 107.696 139.827 0)
+      (effects (font (size 1.27 1.27)) hide)
+    )
+    (property "Value" "GND" (id 1) (at 105.41 139.8269 90)
+      (effects (font (size 1.27 1.27)) (justify right))
+    )
+    (property "Footprint" "" (id 2) (at 101.346 139.827 0)
+      (effects (font (size 1.27 1.27)) hide)
+    )
+    (property "Datasheet" "" (id 3) (at 101.346 139.827 0)
+      (effects (font (size 1.27 1.27)) hide)
+    )
+    (pin "1")
+  )
   (symbol (lib_id "Power_Protection:SP0502BAHT") (at 31.369 51.562 0) (mirror y) (unit 1)
     (in_bom yes) (on_board yes)
-    (property "Reference" "D?" (id 0) (at 32.385 51.181 0)
+    (property "Reference" "D2" (id 0) (at 32.385 51.181 0)
       (effects (font (size 1.27 1.27)) (justify left))
     )
@@
   (symbol (lib_id "AERO_Symbols:Dev_Board_C") (at 121.412 65.532 0) (unit 1)
     (in_bom yes) (on_board yes) (fields_autoplaced)
-    (property "Reference" "U?" (id 0) (at 119.507 29.591 0))
+    (property "Reference" "U1" (id 0) (at 119.507 29.591 0))
     (property "Value" "Dev_Board_C" (id 1) (at 119.507 32.131 0))
     (property "Footprint" "" (id 2) (at 121.412 65.532 0)

Commit message: rcb
Parts:
- U1: footprint (none) -> esp32:ESP32-DevKitC
Connections:
- net PUMP_CTRL: now also U1.30 (GPIO18); no longer U1.24 (ADC2_CH2/*GPIO2)
- net WATER_IN-: now also U1.28 (GPIO17); no longer U1.26 (ADC2_CH0/GPIO4)
- net DAT2: now reaches J7.1 (DAT2)
- net DAT2: now also U1.13 (*MTDI/GPIO12/ADC2_CH5)
- net DAT1: now reaches J7.8 (DAT1)
- net DAT1: now also U1.26 (ADC2_CH0/GPIO4)
- net SD_CS renamed CMD
- net CMD: now also J7.3 (CMD); no longer J7.2 (DAT3/CD)
- net SD_MISO renamed DAT0
- net DAT0: now also U1.24 (ADC2_CH2/*GPIO2); no longer U1.13 (*MTDI/GPIO12/ADC2_CH5)
- net SD_MOSI renamed DAT3
- net DAT3: now also J7.2 (DAT3/CD); no longer J7.3 (CMD)
- net SD_SCK renamed CLK
- no-connect marks 2 -> 0
Changed lines of the file:
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@@
   (junction (at 248.92 136.525) (diameter 0) (color 0 0 0 0)
   )
-  (no_connect (at 101.346 152.527))
-  (no_connect (at 101.346 134.747))
   (wire (pts (xy 61.849 56.642) (xy 84.582 56.642))
     (stroke (width 0) (type default) (color 0 0 0 0))
@@
     (effects (font (size 1.27 1.27)) (justify left bottom))
   )
-  (label "SD_CS" (at 101.346 149.987 0)
-    (effects (font (size 1.27 1.27)) (justify left bottom))
+  (label "DAT2" (at 84.582 69.342 180)
+    (effects (font (size 1.27 1.27)) (justify right bottom))
   )
   (label "CAN_MISO" (at 243.205 136.525 180)
     (effects (font (size 1.27 1.27)) (justify right bottom))
   )
+  (label "DAT0" (at 101.346 137.287 0)
+    (effects (font (size 1.27 1.27)) (justify left bottom))
+  )
+  (label "DAT2" (at 101.346 152.527 0)
+    (effects (font (size 1.27 1.27)) (justify left bottom))
+  )
+  (label "DAT3" (at 101.346 149.987 0)
+    (effects (font (size 1.27 1.27)) (justify left bottom))
+  )
   (label "TEMP_WATER_OUT" (at 243.459 83.566 180)
     (effects (font (size 1.27 1.27)) (justify right bottom))
   )
-  (label "SD_SCK" (at 101.346 142.367 0)
-    (effects (font (size 1.27 1.27)) (justify left bottom))
-  )
-  (label "SD_MISO" (at 84.582 69.342 180)
+  (label "DAT3" (at 84.582 74.422 180)
     (effects (font (size 1.27 1.27)) (justify right bottom))
   )
-  (label "SD_MOSI" (at 101.346 147.447 0)
+  (label "DAT1" (at 101.346 134.747 0)
+    (effects (font (size 1.27 1.27)) (justify left bottom))
+  )
+  (label "TEMP_WATER_IN" (at 154.432 64.262 0)
+    (effects (font (size 1.27 1.27)) (justify left bottom))
+  )
+  (label "CMD" (at 154.432 76.962 0)
     (effects (font (size 1.27 1.27)) (justify left bottom))
   )
@@
     (effects (font (size 1.27 1.27)) (justify left bottom))
   )
-  (label "SD_MOSI" (at 84.582 74.422 180)
+  (label "CLK" (at 101.346 142.367 0)
+    (effects (font (size 1.27 1.27)) (justify left bottom))
+  )
+  (label "CMD" (at 101.346 147.447 0)
+    (effects (font (size 1.27 1.27)) (justify left bottom))
+  )
+  (label "CAN_MOSI" (at 193.675 136.525 0)
+    (effects (font (size 1.27 1.27)) (justify left bottom))
+  )
+  (label "DAT0" (at 154.432 74.422 0)
+    (effects (font (size 1.27 1.27)) (justify left bottom))
+  )
+  (label "TEMP_WATER_OUT" (at 154.432 71.882 0)
+    (effects (font (size 1.27 1.27)) (justify left bottom))
+  )
+  (label "CLK" (at 84.582 66.802 180)
     (effects (font (size 1.27 1.27)) (justify right bottom))
   )
-  (label "CAN_MOSI" (at 193.675 136.525 0)
-    (effects (font (size 1.27 1.27)) (justify left bottom))
-  )
-  (label "SD_SCK" (at 84.582 66.802 180)
-    (effects (font (size 1.27 1.27)) (justify right bottom))
-  )
-  (label "SD_CS" (at 154.432 76.962 0)
-    (effects (font (size 1.27 1.27)) (justify left bottom))
-  )
-  (label "TEMP_WATER_OUT" (at 154.432 71.882 0)
-    (effects (font (size 1.27 1.27)) (justify left bottom))
-  )
-  (label "SD_MISO" (at 101.346 137.287 0)
-    (effects (font (size 1.27 1.27)) (justify left bottom))
-  )
-  (label "TEMP_WATER_IN" (at 154.432 69.342 0)
+  (label "DAT1" (at 154.432 69.342 0)
     (effects (font (size 1.27 1.27)) (justify left bottom))
   )
@@
     (effects (font (size 1.27 1.27)) (justify left))
   )
+  (hierarchical_label "PUMP_CTRL" (shape output) (at 154.432 59.182 0)
+    (effects (font (size 1.27 1.27)) (justify left))
+  )
   (hierarchical_label "WATER_OUT+" (shape input) (at 226.314 78.486 180)
     (effects (font (size 1.27 1.27)) (justify right))
@@
   )
   (hierarchical_label "FAULT_IMD" (shape input) (at 56.769 53.213 0)
-    (effects (font (size 1.27 1.27)) (justify left))
-  )
-  (hierarchical_label "PUMP_CTRL" (shape output) (at 154.432 74.422 0)
     (effects (font (size 1.27 1.27)) (justify left))
   )
@@
     (property "Reference" "U1" (id 0) (at 119.507 29.591 0))
     (property "Value" "Dev_Board_C" (id 1) (at 119.507 32.131 0))
-    (property "Footprint" "" (id 2) (at 121.412 65.532 0)
-      (effects (font (size 1.27 1.27)) hide)
-    )
+    (property "Footprint" "esp32:ESP32-DevKitC" (id 2) (at 121.412 65.532 0)
+      (effects (font (size 1.27 1.27)) hide)
+    )

Commit message: update
Connections:
- net BRAKE_CTRL: now also U1.9 (DAC_1/ADC2_CH8/GPIO25); no longer U1.10 (DAC_2/ADC2_CH9/GPIO26)
- net FAN_CTRL: now also U1.10 (DAC_2/ADC2_CH9/GPIO26); no longer U1.9 (DAC_1/ADC2_CH8/GPIO25)
Changed lines of the file:
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@@
     (effects (font (size 1.27 1.27)) (justify right))
   )
-  (hierarchical_label "BRAKE_CTRL" (shape output) (at 84.582 61.722 180)
+  (hierarchical_label "BRAKE_CTRL" (shape output) (at 84.582 59.182 180)
     (effects (font (size 1.27 1.27)) (justify right))
   )
@@
     (effects (font (size 1.27 1.27)) (justify left))
   )
-  (hierarchical_label "FAN_CTRL" (shape output) (at 84.582 59.182 180)
+  (hierarchical_label "FAN_CTRL" (shape output) (at 84.582 61.722 180)
     (effects (font (size 1.27 1.27)) (justify right))
   )

Commit message: colin
Other:
- note added: "Pull High low is stby"
- note added: "max5039 on car"
- note removed: "STBY logic low is normal mode logic high is receive only"
Changed lines of the file:
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@@
+    (effects (font (size 1.27 1.27)) (justify left bottom))
+  )
+  (text "max5039 on car" (at 209.931 119.38 0)
+    (effects (font (size 1.27 1.27)) (justify left bottom))
+  )
+  (text "Pull High low is stby" (at 175.26 132.588 0)
     (effects (font (size 1.27 1.27)) (justify left bottom))
   )
@@
     (effects (font (size 1.27 1.27) bold italic) (justify left bottom))
   )
-  (text "STBY logic low is normal mode\nlogic high is receive only"
-    (at 219.71 162.56 0)
-    (effects (font (size 1.27 1.27)) (justify left bottom))
-  )
   (label "DAT2" (at 84.582 69.342 180)
