File: Rear-Control-Board/rear-control-board-Design/FuseBank.kicad_sch (KiCad schematic)
At the start: 10 parts

Commit message: pcb Done? check SD
Parts:
- F5: value 2A -> 5A
Connections:
- net REAR_12V renamed BMS_12V
- net SPARE_12V renamed HVB_12
Changed lines of the file:
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@@
     (effects (font (size 1.27 1.27)) (justify left))
   )
-  (hierarchical_label "REAR_12V" (shape output) (at 101.6 85.725 0)
+  (hierarchical_label "BMS_12V" (shape output) (at 101.6 85.725 0)
     (effects (font (size 1.27 1.27)) (justify left))
   )
@@
     (effects (font (size 1.27 1.27)) (justify right))
   )
-  (hierarchical_label "SPARE_12V" (shape output) (at 101.6 98.425 0)
+  (hierarchical_label "HVB_12" (shape output) (at 101.6 98.425 0)
     (effects (font (size 1.27 1.27)) (justify left))
   )
@@
     (in_bom yes) (on_board yes)
     (property "Reference" "F5" (id 0) (at 86.36 83.185 90))
-    (property "Value" "2A" (id 1) (at 81.28 83.185 90))
+    (property "Value" "5A" (id 1) (at 81.28 83.185 90))
     (property "Footprint" "AERO_Footprints:Fuseholder_Blade_Mini_Keystone_3568" (id 2) (at 83.82 83.947 90)
       (effects (font (size 1.27 1.27)) hide)

Commit message: commit
Changed lines of the file:
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@@
   (junction (at 74.93 98.425) (diameter 0) (color 0 0 0 0)
   )
+  (junction (at 99.695 85.725) (diameter 0) (color 0 0 0 0)
+  )
   (junction (at 74.93 60.325) (diameter 0) (color 0 0 0 0)
   )
@@
     (stroke (width 0) (type default) (color 0 0 0 0))
   )
-  (wire (pts (xy 101.6 85.725) (xy 87.63 85.725))
+  (wire (pts (xy 101.6 85.725) (xy 99.695 85.725))
     (stroke (width 0) (type default) (color 0 0 0 0))
   )
@@
     (stroke (width 0) (type default) (color 0 0 0 0))
   )
+  (wire (pts (xy 113.665 88.011) (xy 99.695 88.011))
+    (stroke (width 0) (type default) (color 0 0 0 0))
+  )
   (wire (pts (xy 100.965 104.14) (xy 87.63 104.14))
     (stroke (width 0) (type default) (color 0 0 0 0))
   )
+  (wire (pts (xy 99.695 85.725) (xy 87.63 85.725))
+    (stroke (width 0) (type default) (color 0 0 0 0))
+  )
   (wire (pts (xy 80.01 85.725) (xy 74.93 85.725))
     (stroke (width 0) (type default) (color 0 0 0 0))
@@
   )
   (wire (pts (xy 80.01 66.675) (xy 74.93 66.675))
+    (stroke (width 0) (type default) (color 0 0 0 0))
+  )
+  (wire (pts (xy 99.695 88.011) (xy 99.695 85.725))
     (stroke (width 0) (type default) (color 0 0 0 0))
   )
@@
     (effects (font (size 1.27 1.27) bold italic) (justify left bottom))
   )
+  (global_label "BMS_12V" (shape input) (at 113.665 88.011 0) (fields_autoplaced)
+    (effects (font (size 1.27 1.27)) (justify left))
+    (property "Intersheet References" "${INTERSHEET_REFS}" (id 0) (at 124.3954 87.9316 0)
+      (effects (font (size 1.27 1.27)) (justify left) hide)
+    )
+  )
   (global_label "INT_12V" (shape output) (at 100.965 60.325 0) (fields_autoplaced)

Commit message: colin
Connections:
- net +12V: no longer F9.1
- new net Bat_12: F9.1
Changed lines of the file:
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@@
   (junction (at 74.93 66.675) (diameter 0) (color 0 0 0 0)
   )
-  (junction (at 74.93 104.14) (diameter 0) (color 0 0 0 0)
-  )
   (junction (at 74.93 85.725) (diameter 0) (color 0 0 0 0)
   )
@@
   )
   (wire (pts (xy 74.93 98.425) (xy 74.93 104.14))
-    (stroke (width 0) (type default) (color 0 0 0 0))
-  )
-  (wire (pts (xy 74.93 104.14) (xy 74.93 110.49))
     (stroke (width 0) (type default) (color 0 0 0 0))
   )
@@
     )
   )
+  (global_label "Bat_12" (shape input) (at 74.93 110.49 180) (fields_autoplaced)
+    (effects (font (size 1.27 1.27)) (justify right))
+    (property "Intersheet References" "${INTERSHEET_REFS}" (id 0) (at 66.0744 110.4106 0)
+      (effects (font (size 1.27 1.27)) (justify right) hide)
+    )
+  )
