File: Rear-Control-Board/rear-control-board-Design/rear-control-board.kicad_pcb (KiCad board)
At the start: 2 copper layers, 99.7 x 113 mm, 69 parts, among them J1 Conn_01x23, J2 Conn_01x23, J3 Conn_01x08, J4 JST-B2B-VERT-2PIN, J5 JST-B2B-VERT-2PIN, J6 FTSH-107-01-F-DV-K, K1 T9VV1K15-12S, K2 G5V-2, K3 G5V-2, U1 STM32F413CGUx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

Commit message: pcb Done? check SD
Parts:
- removed C10, C11, C5, C7, C9: 0.1u, Capacitor_SMD:C_0603_1608Metric_Pad1.08x0.95mm_HandSolder
- removed C4: 4.7u, Capacitor_SMD:C_0603_1608Metric_Pad1.08x0.95mm_HandSolder
- removed D8: SP0502BAHT, Package_TO_SOT_SMD:SOT-23
- removed G***: LOGO, AERO_Footprints:AERO_Logo_10x4mm
- removed J6: FTSH-107-01-F-DV-K, Connector_PinHeader_1.27mm:PinHeader_2x07_P1.27mm_Vertical_SMD
- removed JP1: SolderJumper_2_Bridged, Jumper:SolderJumper-2_P1.3mm_Bridged_Pad1.0x1.5mm
- removed K1: T9VV1K15-12S, AERO_Footprints:RELAY_T9VV1K15-12S
- removed R10: 100, Resistor_SMD:R_0603_1608Metric_Pad0.98x0.95mm_HandSolder
- removed U1: STM32F413CGUx, Package_DFN_QFN:QFN-48-1EP_7x7mm_P0.5mm_EP5.6x5.6mm
- removed Y1: CSTNE8M00, AERO_Footprints:Resonator_SMD_muRata_CSTxExxV-3Pin_3.0x1.1mm_HandSoldering
- added D2: SP0502BAHT, Package_TO_SOT_SMD:SOT-23, F.Cu at (34.5, 91.0)
- added Q1: B5584, Package_TO_SOT_SMD:SOT-363_SC-70-6, F.Cu at (181.4, 69.5)
- added Q2: PSMN5R2-60YL, Package_TO_SOT_SMD:LFPAK56, F.Cu at (95.7, 98.4)
- C13, C2, C3, D4, D5, R1, R11, R12, R13, R14, R15, R16, R17, R9: moved to F.Cu
- F5: value 2A -> 5A
- moved R7 137.7 mm to (34.2, 94.5), turned to 0 degrees
- moved H1 130.6 mm to (41.0, 63.0)
- moved R4 126.9 mm to (39.1, 87.9), turned to 0 degrees
- moved D7 125.7 mm to (39.0, 84.5)
- moved J2 123.1 mm to (44.4, 42.4), turned to 0 degrees
- moved F9 120.6 mm to (194.8, 106.7)
- moved R6 119.3 mm to (29.4, 98.9), turned to 0 degrees
- moved D9 118.1 mm to (29.6, 95.5), turned to 0 degrees
- moved D6 116.1 mm to (29.6, 91.0), turned to 0 degrees
- moved U4 115.7 mm to (32.3, 85.5), turned to 0 degrees
- moved U3 114.9 mm to (32.1, 63.1)
- moved J1 114.5 mm to (44.4, 22.5)
- moved F2 114.1 mm to (194.8, 115.0)
- moved F1 107.1 mm to (159.7, 115.0)
- moved F5 101.6 mm to (177.2, 106.7)
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Connections:
- D4 pad 2: /FAULT_LATCHER/BMS_SWITCH -> /FAULT_LATCHER/BMS_IND
- D6 pad 1: /FAULT_LATCHER/BMS_SWITCH -> /SUSPENSION_R
- D6 pad 2: /Controller/FAULT_IMD -> /SUSPENSION_L
- D7 pad 1: /SUSPENSION_R -> /FAULT_LATCHER/BMS_IND
- D7 pad 2: /SUSPENSION_L -> /Controller/FAULT_IMD
- F5 pad 2: /REAR_12V -> /FuseBank/BMS_12V
- J4 pad 1: /FAULT_LATCHER/BMS_SWITCH -> /FAULT_LATCHER/BMS_IND
- K2 pad 1: /FAULT_LATCHER/BMS_SWITCH -> /FAULT_LATCHER/BMS_IND
- K2 pad 8: /FAULT_LATCHER/BMS_SWITCH -> /FAULT_LATCHER/BMS_IND
- R3 pad 2: /FAULT_LATCHER/BMS_SWITCH -> /FAULT_LATCHER/BMS_IND
- U4 pad 1: /Controller/CAN_TX -> /Controller/CAN_MISO
- U4 pad 4: /Controller/CAN_RX -> /Controller/CAN_MOSI
Routing:
- net +3V3: track 236.8 -> 0.00 mm, vias 10 -> 0
- net /REAR_12V: track 169.1 -> 0.00 mm
- net /FAULT_IMD: track 133.4 -> 0.00 mm
- net /BRB_RTN: track 129.0 -> 0.00 mm
- net /FAULT_BMS: track 128.7 -> 0.00 mm
- net /FuseBank/BRB_LOOP: track 99.8 -> 0.00 mm
- net /Controller/PUMP_CTRL: track 97.4 -> 0.00 mm, vias 1 -> 0
- net /Controller/BRAKE_CTRL: track 97.3 -> 0.00 mm, vias 1 -> 0
- net INT_12V: track 97.2 -> 0.00 mm
- net /Controller/FAN_CTRL: track 89.1 -> 0.00 mm, vias 1 -> 0
- net /SSOK: track 75.2 -> 0.00 mm
- net /FuseBank/FRONT_12V: track 73.6 -> 0.00 mm
- net /FAULT_LATCHER/BMS_SWITCH: track 68.6 -> 0.00 mm
- net /BRAKE_12V: track 55.7 -> 0.00 mm
- net /CAN_N: track 46.8 -> 0.00 mm
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- removed copper zone on B.Cu, net +12V
- removed copper zone on F.Cu, net +12V
- removed copper zone on B.Cu, net /BATT_12V
- removed copper zone on F.Cu, net /BATT_12V
- removed copper zone on B.Cu, net /BRAKE_CTRL_12V
- removed copper zone on F.Cu, net /BRAKE_CTRL_12V
- removed copper zone on B.Cu, net /DCDC_IN
- removed copper zone on F.Cu, net /DCDC_IN
- removed copper zone on B.Cu, net /FAN_12V
- removed copper zone on F.Cu, net /FAN_12V
- removed copper zone on B.Cu, net /FAN_CTRL_12V
- removed copper zone on F.Cu, net /FAN_CTRL_12V
- removed copper zone on B.Cu, net /FuseBank/RINE_12V
- removed copper zone on F.Cu, net /FuseBank/RINE_12V
- removed copper zone on B.Cu, net /FuseBank/SPARE_12V
- removed copper zone on F.Cu, net /FuseBank/SPARE_12V
- removed copper zone on B.Cu, net /PUMP_12V
- removed copper zone on F.Cu, net /PUMP_12V
- removed copper zone on B.Cu, net /PUMP_CTRL_12V
- removed copper zone on F.Cu, net /PUMP_CTRL_12V
- removed copper zone on B.Cu, net /charge-controller/dcdc_fuse
- removed copper zone on F.Cu, net /charge-controller/dcdc_fuse
- removed copper zone on B.Cu, net GND
- removed copper zone on F.Cu, net GND
Other:
- board outline removed
- board text removed: "BMS"
- board text removed: "DCDC"
- board text removed: "G.Spearing 22.032"
- board text removed: "IMD"
- board text removed: "M3 Holes"
- board text removed: "RCB"
- board text removed: "SSOK"

Commit message: rcb
Parts:
- removed C6: 10u, Capacitor_SMD:C_0603_1608Metric_Pad1.08x0.95mm_HandSolder
- removed R1, R14, R16: 20k, Resistor_SMD:R_0603_1608Metric_Pad0.98x0.95mm_HandSolder
- removed R15, R9: 50k, Resistor_SMD:R_0603_1608Metric_Pad0.98x0.95mm_HandSolder
- removed R17: 200k, Resistor_SMD:R_0603_1608Metric_Pad0.98x0.95mm_HandSolder
- removed U3: LDL1117S33R, Package_TO_SOT_SMD:SOT-223-3_TabPin2
- removed U5, U6, U7: BV1HAL45EFJ, Package_SO:HTSOP-8-1EP_3.9x4.9mm_P1.27mm_EP2.4x3.2mm_ThermalVias
- added C4: 10uF, Capacitor_SMD:C_0603_1608Metric_Pad1.08x0.95mm_HandSolder, F.Cu at (216.5, 26.3)
- added D8: LED, LED_SMD:LED_0603_1608Metric_Pad1.05x0.95mm_HandSolder, F.Cu at (204.4, 31.8)
- added J6: Conn_01x02, Connector_JST:JST_NV_B02P-NV_1x02_P5.00mm_Vertical, F.Cu at (114.8, 125.5)
- added J7: Micro_SD_Card, Connector_Card:microSD_HC_Wuerth_693072010801, F.Cu at (168.7, 76.8)
- added K1: T9VV1K15-12S, AERO_Footprints:RELAY_T9VV1K15-12S, F.Cu at (107.2, 83.2)
- added Q3: PSMN5R2-60YL, Package_TO_SOT_SMD:LFPAK56, F.Cu at (89.8, 108.0)
- added Q4: PSMN5R2-60YL, Package_TO_SOT_SMD:LFPAK56, F.Cu at (90.0, 115.5)
- added R10: 470, Resistor_SMD:R_0603_1608Metric_Pad0.98x0.95mm_HandSolder, F.Cu at (234.8, 30.0)
- added U1: Dev_Board_C, esp32:ESP32-DevKitC, F.Cu at (181.9, 94.0)
- added U2: TS2940CP33 ROG, Package_TO_SOT_SMD:TO-252-2, F.Cu at (164.8, 55.0)
- C1: value .1u -> 10uF
- D1: value LED -> TS4148C RZG; footprint LED_SMD:LED_0603_1608Metric_Pad1.05x0.95mm_HandSolder -> Diode_SMD:D_0603_1608Metric_Pad1.05x0.95mm_HandSolder
- moved R6 226.3 mm to (243.2, 25.0)
- moved D9 225.4 mm to (250.5, 50.5)
- moved R7 220.1 mm to (248.4, 43.5)
- moved D2 220.1 mm to (248.6, 40.0)
- moved D6 208.7 mm to (236.5, 63.5)
- moved R4 202.8 mm to (238.9, 52.7)
- moved D7 202.8 mm to (238.8, 49.2)
- moved D1 165.5 mm to (216.6, 23.7)
- moved C12 164.9 mm to (207.8, 67.8)
- moved C8 164.9 mm to (207.8, 70.3)
- moved C1 151.9 mm to (208.8, 31.8)
- moved R2 147.7 mm to (213.1, 31.8)
- moved R11 133.3 mm to (227.2, 50.2)
- moved R12 133.3 mm to (227.2, 46.2)
- moved C3 133.3 mm to (235.7, 37.3)
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Connections:
- net /FuseBank/SPARE_12V renamed /FuseBank/HVB_12
- C12 pad 1: +3V3 -> VDD
- C13 pad 1: /BRAKE_12V -> /FAN_RTRN_12V
- C2 pad 1: /FAN_12V -> /PUMP_RTRN_12V
- C3 pad 1: /PUMP_12V -> /BRAKE_RTRN_12V
- C8 pad 1: +3V3 -> VDD
- D1 pad 1: GND -> INT_12V
- D1 pad 2: Net-(D1-Pad2) -> GND
- J1 pad 2: /PUMP_CTRL_12V -> /PUMP_12V
- J1 pad 3: /FAN_CTRL_12V -> /FAN_12V
- J1 pad 4: /BRAKE_CTRL_12V -> /BRAKE_12V
- J2 pad 18: +3V3 -> VDD
- J2 pad 19: +3V3 -> VDD
- J2 pad 20: +3V3 -> VDD
- J2 pad 21: +3V3 -> VDD
- J2 pad 22: +3V3 -> VDD
- J2 pad 23: +3V3 -> VDD
- J2 pad 3: unconnected-(J2-Pad3) -> /BRAKE_RTRN_12V
- J2 pad 4: unconnected-(J2-Pad4) -> /FAN_RTRN_12V
- J2 pad 5: unconnected-(J2-Pad5) -> /PUMP_RTRN_12V
- J3 pad 1: /REAR_12V -> unconnected-(J3-Pad1)
- J3 pad 6: /CAN_N -> unconnected-(J3-Pad6)
- J3 pad 7: /CAN_P -> unconnected-(J3-Pad7)
- Q1 pad 1: +3V3 -> VDD
- Q2 pad 4: Net-(Q2-Pad4) -> Net-(R13-Pad2)
- Q2 pad 5: /PUMP_CTRL_12V -> /FAN_RTRN_12V
- R2 pad 1: Net-(D1-Pad2) -> VDD
- R2 pad 2: +3V3 -> Net-(D8-Pad2)
- R3 pad 1: +3V3 -> VDD
- U4 pad 3: +3V3 -> VDD
- U4 pad 5: +3V3 -> VDD

Commit message: commit
Parts:
- removed Q1: B5584, Package_TO_SOT_SMD:SOT-363_SC-70-6
- added D10: FERD20M60ST, Package_TO_SOT_THT:TO-220-3_Vertical, F.Cu at (155.2, 67.9)
- added D11: FERD20M60ST, Package_TO_SOT_THT:TO-220-3_Vertical, F.Cu at (142.0, 67.7)
- added D12: FERD20M60ST, Package_TO_SOT_THT:TO-220-3_Vertical, F.Cu at (130.7, 67.7)
- D3, D7, J7, R10, R5, R8: moved to B.Cu
- moved R6 142.7 mm to (150.2, 133.2), turned to 180 degrees
- moved J2 138.5 mm to (210.5, 84.1), turned to 180 degrees
- moved D9 132.2 mm to (150.2, 136.8), turned to 90 degrees
- moved C4 119.9 mm to (112.2, 85.5), turned to 90 degrees
- moved D1 119.4 mm to (112.2, 81.7), turned to -90 degrees
- moved R7 113.2 mm to (159.0, 113.0), turned to 180 degrees
- moved F3 111.5 mm to (106.0, 131.4), turned to 180 degrees
- moved R8 109.6 mm to (131.4, 121.5), turned to 90 degrees
- moved D2 105.9 mm to (195.8, 131.8)
- moved R2 103.3 mm to (124.5, 84.7), turned to 90 degrees
- moved C1 100.3 mm to (118.7, 76.0)
- moved D5 100.2 mm to (143.2, 113.0), turned to 90 degrees
- moved R5 100.1 mm to (136.2, 121.5), turned to -90 degrees
- moved F8 99.4 mm to (106.0, 122.2), turned to 180 degrees
- moved R4 95.7 mm to (159.0, 105.5), turned to 180 degrees
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Connections:
- F10 pad 2: /FuseBank/TSV -> /TSV
- F5 pad 2: /FuseBank/BMS_12V -> BMS_12V
- J1 pad 12: /BATT_12V -> /FAULT_BMS
- J1 pad 13: /BATT_12V -> /BRB_RTN
- J1 pad 20: /BRB_RTN -> /TSV
- J1 pad 22: /FAULT_BMS -> /DCDC_IN
- J1 pad 23: /FuseBank/TSV -> /DCDC_IN
- J1 pad 7: /DCDC_IN -> /BATT_12V
- J1 pad 8: /DCDC_IN -> /BATT_12V
- J2 pad 12: unconnected-(J2-Pad12) -> BMS_12V
- J2 pad 15: /WATER_IN- -> /WATER_OUT-
- J2 pad 8: /WATER_OUT- -> /WATER_IN-
Routing:
- net VDD: track 0.00 -> 230.2 mm, vias 0 -> 1
- net /BRB_RTN: track 0.00 -> 127.5 mm
- net /TSV: track 0.00 -> 117.5 mm, vias 0 -> 1
- net INT_12V: track 0.00 -> 81.9 mm
- net /Controller/FAULT_IMD: track 0.00 -> 59.2 mm
- net /FAULT_IMD: track 0.00 -> 58.4 mm
- net /FAULT_LATCHER/IMD_SWITCH: track 0.00 -> 36.4 mm
- net /FAULT_LATCHER/BMS_IND: track 0.00 -> 34.7 mm
- net /CAN_P: track 0.00 -> 33.2 mm
- net /CAN_N: track 0.00 -> 31.9 mm
- net /BRAKE_12V: track 0.00 -> 28.9 mm
- net /SSOK: track 0.00 -> 22.6 mm
- net /Controller/CAN_MOSI: track 0.00 -> 20.6 mm, vias 0 -> 1
- net /charge-controller/dcdc_fuse: track 0.00 -> 19.2 mm
- net /Controller/CAN_MISO: track 0.00 -> 14.5 mm
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- added copper zone on B.Cu, net +12V
- added copper zone on B.Cu, net /BATT_12V
- added copper zone on B.Cu, net /DCDC_IN

Commit message: update
Parts:
- removed R10: 470, Resistor_SMD:R_0603_1608Metric_Pad0.98x0.95mm_HandSolder
- removed R11, R12, R13: 1.5K, Resistor_SMD:R_0603_1608Metric_Pad0.98x0.95mm_HandSolder
- D2, D6: moved to B.Cu
- J7: moved to F.Cu
- moved Q3 78.5 mm to (80.0, 87.3)
- moved C3 77.7 mm to (76.2, 86.8)
- moved D10 71.5 mm to (86.1, 86.3), turned to -90 degrees
- moved C13 68.0 mm to (75.8, 73.5), turned to 90 degrees
- moved Q2 67.9 mm to (80.0, 77.8)
- moved H1 64.6 mm to (28.0, 50.0)
- moved H2 64.6 mm to (36.0, 50.0)
- moved C2 57.2 mm to (76.2, 66.0)
- moved Q4 57.1 mm to (80.2, 66.3)
- moved D11 56.3 mm to (86.1, 74.7), turned to -90 degrees
- moved D2 51.0 mm to (170.1, 87.7), turned to 180 degrees
- moved D12 45.0 mm to (85.9, 63.3), turned to -90 degrees
- moved D6 44.2 mm to (179.9, 85.8), turned to 180 degrees
- moved F8 34.2 mm to (106.0, 88.0)
- moved J7 30.8 mm to (188.2, 157.2), turned to 0 degrees
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Connections:
- net /FAULT_LATCHER/BMS_IND renamed /FAULT_LATCHER/BMS_SWITCH
- F3 pad 2: /FuseBank/RINE_12V -> /RINE_12
- F4 pad 2: /FuseBank/FRONT_12V -> /FRONT_12
- F7 pad 2: /FuseBank/HVB_12 -> /HVB_12
- F9 pad 2: /FuseBank/BRB_LOOP -> /BRB_LOOP
- J1 pad 1: /FuseBank/HVB_12 -> /FAN_RTRN_12V
- J1 pad 12: /FAULT_BMS -> /BATT_12V
- J1 pad 13: /BRB_RTN -> /BATT_12V
- J1 pad 14: /DCDC_IN -> /BATT_12V
- J1 pad 15: /DCDC_IN -> /BATT_12V
- J1 pad 16: /FuseBank/FRONT_12V -> /PUMP_RTRN_12V
- J1 pad 17: /FuseBank/BRB_LOOP -> GND
- J1 pad 19: GND -> /FRONT_12
- J1 pad 2: /PUMP_12V -> /FAN_12V
- J1 pad 20: /TSV -> /DCDC_IN
- J1 pad 21: /FAULT_IMD -> /DCDC_IN
- J1 pad 3: /FAN_12V -> /BRAKE_RTRN_12V
- J1 pad 5: /BATT_12V -> /HVB_12
- J1 pad 6: /BATT_12V -> BMS_12V
- J1 pad 7: /BATT_12V -> /FAULT_BMS
- J1 pad 8: /BATT_12V -> /FAULT_IMD
- J1 pad 9: /FuseBank/RINE_12V -> /PUMP_12V
- J2 pad 12: BMS_12V -> unconnected-(J2-Pad12)
- J2 pad 3: /BRAKE_RTRN_12V -> unconnected-(J2-Pad3)
- J2 pad 4: /FAN_RTRN_12V -> unconnected-(J2-Pad4)
- J2 pad 5: /PUMP_RTRN_12V -> unconnected-(J2-Pad5)
- J3 pad 1: unconnected-(J3-Pad1) -> /BRB_LOOP
- J3 pad 6: unconnected-(J3-Pad6) -> /RINE_12
- J3 pad 7: unconnected-(J3-Pad7) -> /TSV
- J3 pad 8: GND -> /BRB_RTN
- Q2 pad 4: Net-(Q2-Pad4) -> /Controller/BRAKE_CTRL
- Q3 pad 4: Net-(Q3-Pad4) -> /Controller/PUMP_CTRL
- Q4 pad 4: Net-(Q4-Pad4) -> /Controller/FAN_CTRL
- U1 pad 10: /Controller/BRAKE_CTRL -> /Controller/FAN_CTRL
- U1 pad 9: /Controller/FAN_CTRL -> /Controller/BRAKE_CTRL
Routing:
- net /Controller/BRAKE_CTRL: track 0.00 -> 127.4 mm, vias 0 -> 1
- net /Controller/FAN_CTRL: track 0.00 -> 127.1 mm, vias 0 -> 1
- net /Controller/PUMP_CTRL: track 0.00 -> 94.2 mm, vias 0 -> 1
- net /TSV: track 117.5 -> 36.7 mm, vias 1 -> 0
- net /FAULT_BMS: track 0.00 -> 62.6 mm
- net /Controller/FAULT_IMD: track 59.2 -> 5.29 mm
- net /HVB_12: track 0.00 -> 53.0 mm
- net /BRB_LOOP: track 0.00 -> 47.6 mm
- net BMS_12V: track 0.00 -> 47.0 mm
- net /WATER_IN-: track 0.00 -> 45.5 mm
- net /FRONT_12: track 0.00 -> 43.3 mm
- net /WATER_OUT-: track 0.00 -> 41.2 mm
- net INT_12V: track 81.9 -> 41.1 mm
- net /BRAKE_RTRN_12V: track 0.00 -> 30.2 mm
- net VDD: track 230.2 -> 251.5 mm, vias 1 -> 0
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- added copper zone on B.Cu, net /FAN_12V
- added copper zone on F.Cu, net /FAN_RTRN_12V
- added copper zone on B.Cu, net /PUMP_12V
- added copper zone on F.Cu, net /PUMP_RTRN_12V
- added copper zone on B.Cu, net /RINE_12

Commit message: DONE!!!!!
Parts:
- D2, D6: moved to F.Cu
- moved D7 32.7 mm to (182.2, 121.8)
- moved D6 11.3 mm to (169.8, 80.8), turned to -90 degrees
- moved D2 9.60 mm to (163.5, 80.7), turned to -90 degrees
Connections:
- J2 pad 13: /WHEEL_L -> unconnected-(J2-Pad13)
- J2 pad 14: /SUSPENSION_L -> unconnected-(J2-Pad14)
- J2 pad 4: unconnected-(J2-Pad4) -> /SUSPENSION_R
- J2 pad 5: unconnected-(J2-Pad5) -> /SUSPENSION_L
- J2 pad 7: /SUSPENSION_R -> /WHEEL_L
Routing:
- net /Controller/DAT0: track 0.00 -> 87.9 mm, vias 0 -> 1
- net /Controller/DAT1: track 0.00 -> 70.7 mm, vias 0 -> 3
- net /WHEEL_R: track 0.00 -> 68.9 mm
- net /Controller/CLK: track 0.00 -> 68.2 mm, vias 0 -> 1
- net /WHEEL_L: track 4.12 -> 72.3 mm
- net /Controller/CMD: track 0.00 -> 65.6 mm, vias 0 -> 2
- net /SUSPENSION_L: track 0.00 -> 63.9 mm
- net /SUSPENSION_R: track 0.00 -> 60.5 mm
- net /Controller/DAT3: track 0.00 -> 56.3 mm, vias 0 -> 1
- net /FAULT_LATCHER/BMS_SWITCH: track 34.7 -> 90.7 mm, vias 0 -> 1
- net /Controller/FAULT_IMD: track 5.29 -> 60.4 mm
- net /Controller/DAT2: track 0.00 -> 51.0 mm, vias 0 -> 1
- net INT_12V: track 41.1 -> 72.7 mm, vias 0 -> 2
- net GND: vias 0 -> 17
- added copper zone on B.Cu, net GND
- added copper zone on F.Cu, net GND
Other:
- board outline added: 139.1 x 102.8 mm

Commit message: V1 with all Gerbers
Routing:
- net +12V: track 0.00 -> 95.6 mm
- net /DCDC_IN: track 0.00 -> 50.5 mm
- net /PUMP_RTRN_12V: track 0.00 -> 34.5 mm
- net /FAN_RTRN_12V: track 0.00 -> 12.4 mm
- net /BATT_12V: track 0.00 -> 11.9 mm
- net /RINE_12: track 0.00 -> 3.35 mm
- net /PUMP_12V: track 0.00 -> 3.20 mm
- net GND: vias 17 -> 16
Changed lines of the file:
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@@
       (drillshape 0)
       (scaleselection 1)
-      (outputdirectory "RCB_Gerber/")
+      (outputdirectory "../../BOARD GERBER/V1/RCB/")
     )
   )
@@
     (fp_line (start -2.45 3.4) (end 4.95 3.4) (layer "F.Fab") (width 0.1))
     (pad "" np_thru_hole circle (at -1.6 2 90) (size 1.2 1.2) (drill 1.2) (layers *.Cu *.Mask))
-    (pad "1" thru_hole roundrect (at 0 0 90) (size 1.7 2) (drill 1) (layers *.Cu *.Mask) (roundrect_rratio 0.147059)
+    (pad "1" thru_hole roundrect (at 0 0 90) (size 1.7 2) (drill 1) (layers *.Cu *.Mask) (roundrect_rratio 0.1470588235)
       (net 67 "/FAULT_LATCHER/BMS_SWITCH") (pinfunction "Pin_1") (pintype "passive"))
     (pad "2" thru_hole oval (at 2.5 0 90) (size 1.7 2) (drill 1) (layers *.Cu *.Mask)
@@
     (fp_line (start -2.45 3.4) (end 4.95 3.4) (layer "F.Fab") (width 0.1))
     (pad "" np_thru_hole circle (at -1.6 2 270) (size 1.2 1.2) (drill 1.2) (layers *.Cu *.Mask))
-    (pad "1" thru_hole roundrect (at 0 0 270) (size 1.7 2) (drill 1) (layers *.Cu *.Mask) (roundrect_rratio 0.147059)
+    (pad "1" thru_hole roundrect (at 0 0 270) (size 1.7 2) (drill 1) (layers *.Cu *.Mask) (roundrect_rratio 0.1470588235)
       (net 3 "INT_12V") (pinfunction "Pin_1") (pintype "passive"))
     (pad "2" thru_hole oval (at 2.5 0 270) (size 1.7 2) (drill 1) (layers *.Cu *.Mask)
@@
     (fp_line (start -2.5 -3.7) (end -2.5 4.8) (layer "F.Fab") (width 0.1))
     (fp_line (start -2.5 -1) (end -1.5 0) (layer "F.Fab") (width 0.1))
-    (pad "1" thru_hole roundrect (at 0 0 180) (size 2.7 2.7) (drill 1.7) (layers *.Cu *.Mask) (roundrect_rratio 0.092593)
+    (pad "1" thru_hole roundrect (at 0 0 180) (size 2.7 2.7) (drill 1.7) (layers *.Cu *.Mask) (roundrect_rratio 0.09259296296)
       (net 19 "/CAN_P") (pinfunction "Pin_1") (pintype "passive"))
     (pad "2" thru_hole circle (at 5 0 180) (size 2.7 2.7) (drill 1.7) (layers *.Cu *.Mask)
@@
   (via (at 190.5 153) (size 0.8) (drill 0.4) (layers "F.Cu" "B.Cu") (free) (net 1))
   (via (at 131 131) (size 0.8) (drill 0.4) (layers "F.Cu" "B.Cu") (free) (net 1))
-  (via (at 89.5 128.75) (size 0.8) (drill 0.4) (layers "F.Cu" "B.Cu") (free) (net 1))
   (via (at 110.5 78.25) (size 0.8) (drill 0.4) (layers "F.Cu" "B.Cu") (free) (net 1))
   (via (at 177.5 128.75) (size 0.8) (drill 0.4) (layers "F.Cu" "B.Cu") (free) (net 1))
@@
   (via (at 113.25 112.25) (size 0.8) (drill 0.4) (layers "F.Cu" "B.Cu") (free) (net 1))
   (via (at 150.25 136.75) (size 0.8) (drill 0.4) (layers "F.Cu" "B.Cu") (free) (net 1))
+  (segment (start 80.15 65.85) (end 78.87298 64.57298) (width 3.175) (layer "F.Cu") (net 2))
+  (segment (start 82.689297 63.310703) (end 84.748777 63.315161) (width 3.175) (layer "F.Cu") (net 2))
+  (segment (start 61.5875 69.566094) (end 61.5875 77.25) (width 3.175) (layer "F.Cu") (net 2))
+  (segment (start 80.15 65.85) (end 82.689297 63.310703) (width 3.175) (layer "F.Cu") (net 2))
+  (segment (start 78.87298 64.57298) (end 66.580614 64.57298) (width 3.175) (layer "F.Cu") (net 2))
+  (segment (start 66.580614 64.57298) (end 61.5875 69.566094) (width 3.175) (layer "F.Cu") (net 2))
   (segment (start 117.8625 75.975) (end 116.975 75.975) (width 0.635) (layer "F.Cu") (net 3))
   (segment (start 141.9175 99.013615) (end 138.4575 99.013615) (width 0.635) (layer "F.Cu") (net 3))
@@
   (segment (start 131.5 92.25) (end 117.775 78.525) (width 0.635) (layer "B.Cu") (net 3))
   (segment (start 117.775 78.525) (end 116.445 78.525) (width 0.635) (layer "B.Cu") (net 3))
+  (segment (start 105.96 137.905) (end 114.625 146.57) (width 3.175) (layer "B.Cu") (net 4))
+  (segment (start 105.96 70.7) (end 105.96 137.905) (width 3.175) (layer "B.Cu") (net 4))
+  (segment (start 114.04 70.7) (end 105.96 70.7) (width 3.175) (layer "B.Cu") (net 4))
+  (segment (start 105.96 67.3) (end 114.04 67.3) (width 3.175) (layer "B.Cu") (net 4))
+  (segment (start 65.5875 103.25) (end 65.5875 91.63892) (width 3.175) (layer "B.Cu") (net 6))
+  (segment (start 65.5875 91.63892) (end 65.39304 91.44446) (width 3.175) (layer "B.Cu") (net 6))
   (segment (start 141.75 110.001115) (end 148.7175 110.001115) (width 0.635) (layer "F.Cu") (net 7))
   (segment (start 136.34 113.376115) (end 138.375 113.376115) (width 0.635) (layer "F.Cu") (net 7))
@@
   (segment (start 135.122989 112.159104) (end 119.777011 112.159104) (width 0.635) (layer "B.Cu") (net 7))
   (segment (start 136.375 116.425) (end 136.375 113.411115) (width 0.635) (layer "B.Cu") (net 7))
+  (segment (start 96.04 67.3) (end 96.04 70.502491) (width 3.175) (layer "F.Cu") (net 8))
   (segment (start 96.04 87.95) (end 94.45 87.95) (width 2.54) (layer "B.Cu") (net 9))
   (segment (start 70.0325 88.805) (end 86.095 88.805) (width 2.54) (layer "B.Cu") (net 9))
@@
   (segment (start 80 86.85) (end 80.585 86.265) (width 2.54) (layer "F.Cu") (net 10))
   (segment (start 88.56452 87.801767) (end 87.027753 86.265) (width 2.54) (layer "F.Cu") (net 10))
+  (segment (start 60.54 94.2975) (end 61.5875 93.25) (width 3.175) (layer "B.Cu") (net 11))
+  (segment (start 60.54 139.95) (end 60.54 136.55) (width 3.175) (layer "B.Cu") (net 11))
+  (segment (start 60.54 139.95) (end 60.54 94.2975) (width 3.175) (layer "B.Cu") (net 11))
   (segment (start 69.5875 101.25) (end 71.444511 99.392989) (width 0.635) (layer "F.Cu") (net 12))
   (segment (start 71.444511 99.392989) (end 122.838126 99.392989) (width 0.635) (layer "F.Cu") (net 12))
@@
   (segment (start 149.615 126.491983) (end 149.615 125.775) (width 0.635) (layer "F.Cu") (net 21))
   (segment (start 121.65 87.75) (end 118.725 84.825) (width 2.54) (layer "F.Cu") (net 21))
+  (segment (start 69.6525 77.315) (end 69.5875 77.25) (width 3.175) (layer "F.Cu") (net 22))
+  (segment (start 80 77.315) (end 69.6525 77.315) (width 3.175) (layer "F.Cu") (net 22))
+  (segment (start 80 77.315) (end 78.065 77.315) (width 3.175) (layer "F.Cu") (net 22))
   (segment (start 124.475 80.35) (end 124.475 83.8125) (width 0.635) (layer "F.Cu") (net 23))
   (segment (start 136.05 123.79) (end 136.05 122.45) (width 0.635) (layer "F.Cu") (net 24))
@@
   (segment (start 82.1375 109.8) (end 69.5875 97.25) (width 2.54) (layer "B.Cu") (net 60))
   (segment (start 96.04 113.2) (end 85.5375 113.2) (width 2.54) (layer "B.Cu") (net 60))
+  (segment (start 115.96 131.45) (end 115.96 128.22078) (width 3.175) (layer "B.Cu") (net 62))
+  (segment (start 115.96 128.22078) (end 115.87461 128.13539) (width 3.175) (layer "B.Cu") (net 62))
   (segment (start 115.96 122.2) (end 115.96 123.8975) (width 2.54) (layer "B.Cu") (net 63))
   (segment (start 115.96 123.8975) (end 146 153.9375) (width 2.54) (layer "B.Cu") (net 63))

Commit message: colin
Parts:
- moved H1 157.8 mm to (182.0, 84.5)
- moved H2 108.1 mm to (70.2, 152.5)
Changed lines of the file:
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@@
   )
   (footprint "MountingHole:MountingHole_3.2mm_M3" (layer "F.Cu")
-    (at 35.95 50)
+    (at 70.25 152.5)
     (descr "Mounting Hole 3.2mm, no annular, M3")
     (tags "mounting hole 3.2mm no annular m3")
@@
   )
   (footprint "MountingHole:MountingHole_3.2mm_M3" (layer "F.Cu")
-    (at 28 50)
+    (at 182 84.5)
     (descr "Mounting Hole 3.2mm, no annular, M3")
     (tags "mounting hole 3.2mm no annular m3")
