File: Rear-Control-Board/rear-control-board-Design/rear-control-board.kicad_sch (KiCad schematic)
At the start: 11 parts, among them J1 Conn_01x23, J2 Conn_01x23, J3 Conn_01x08, K1 T9VV1K15-12S, U3 LDL1117S33R

Commit message: pcb Done? check SD
Parts:
- removed C6: 10u, Capacitor_SMD:C_0603_1608Metric_Pad1.08x0.95mm_HandSolder, symbol Device:C
- removed D1: LED, LED_SMD:LED_0603_1608Metric_Pad1.05x0.95mm_HandSolder, symbol Device:LED
- removed U3: LDL1117S33R, Package_TO_SOT_SMD:SOT-223-3_TabPin2, symbol Regulator_Linear:LD1117S33TR_SOT223
- added C4: 10uF, Capacitor_SMD:C_0603_1608Metric_Pad1.08x0.95mm_HandSolder, symbol Device:C
- added D1: TS4148C RZG, Diode_SMD:D_0603_1608Metric_Pad1.05x0.95mm_HandSolder, symbol Device:D
- added D8: LED, LED_SMD:LED_0603_1608Metric_Pad1.05x0.95mm_HandSolder, symbol Device:LED
- added J6: Conn_01x02, symbol Connector_Generic:Conn_01x02
- added U2: TS2940CP33 ROG, Package_TO_SOT_SMD:TO-252-2, symbol Regulator_Linear:NCP1117-5.0_TO252
- C1: value .1u -> 10uF
Connections:
- net BRAKE_CTRL_12V is gone; now on net BRAKE_12V: J1.4 (Pin_4)
- net FAN_CTRL_12V is gone; now on net FAN_12V: J1.3 (Pin_3)
- net PUMP_CTRL_12V is gone; now on net PUMP_12V: J1.2 (Pin_2)
- net BRB_RTN: now also K1.1
- net CAN_N: now also J6.2 (Pin_2); no longer J3.6 (Pin_6)
- net CAN_P: now also J6.1 (Pin_1); no longer J3.7 (Pin_7)
- net GND: now also C4.2, D1.2 (A), D8.1 (K), U2.1 (GND)
- net INT_12V: now also D1.1 (K), U2.3 (VI)
- net REAR_12V: no longer J3.1 (Pin_1)
- net SSOK: no longer K1.1
- net BRAKE_RTRN_12V: now reaches J2.3 (Pin_3)
- net FAN_RTRN_12V: now reaches J2.4 (Pin_4)
- net PUMP_RTRN_12V: now reaches J2.5 (Pin_5)
- net VDD: now reaches R2.1
- net VDD: now also J2.18 (Pin_18), J2.19 (Pin_19), J2.20 (Pin_20), J2.21 (Pin_21), J2.22 (Pin_22), J2.23 (Pin_23), C4.1, U2.2 (VO)
- removed net +3V3: J2.18 (Pin_18), J2.19 (Pin_19), J2.20 (Pin_20), J2.21 (Pin_21), J2.22 (Pin_22), J2.23 (Pin_23), R2.2
- net FuseBank/SPARE_12V renamed FuseBank/HVB_12
- new net: D8.2 (A), R2.2
Other:
- sheet FET_OUTPUT ports: added none; removed BRAKE_OUT, FAN_OUT, PUMP_OUT
- sheet FuseBank ports: added HVB_12; removed SPARE_12V
- note added: "CAN comes from Rinehart goes to front board"
- note added: "CAN test point"
- note removed: "BMS"
- note removed: "BRB_RTN"
- note removed: "CAN and 12V HVB power"
- note removed: "CAN comes from Rinehart goes to HVB"
- note removed: "DCB"
- note removed: "Footprint is wrong not far enough horizontal hits board edge"
- note removed: "GND to sensors"
- note removed: "HVB not rinehart"
- note removed: "NOT SSOK"
- note removed: "To Other Connector"
- note removed: "to HVB"

Commit message: rcb
Parts:
- J6: footprint (none) -> Connector_JST:JST_NV_B02P-NV_1x02_P5.00mm_Vertical
- K1: footprint AERO-footprints:RELAY_T9VV1K15-12S -> AERO_Footprints:RELAY_T9VV1K15-12S
Changed lines of the file:
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@@
     (property "Reference" "K1" (id 0) (at 216.535 136.0932 90))
     (property "Value" "T9VV1K15-12S" (id 1) (at 216.535 138.4046 90))
-    (property "Footprint" "AERO-footprints:RELAY_T9VV1K15-12S" (id 2) (at 215.265 139.065 0)
+    (property "Footprint" "AERO_Footprints:RELAY_T9VV1K15-12S" (id 2) (at 215.265 139.065 0)
       (effects (font (size 1.27 1.27)) (justify left) hide)
     )
@@
     (property "Reference" "J6" (id 0) (at 65.405 183.388 0))
     (property "Value" "Conn_01x02" (id 1) (at 65.405 185.928 0))
-    (property "Footprint" "" (id 2) (at 65.405 192.659 0)
+    (property "Footprint" "Connector_JST:JST_NV_B02P-NV_1x02_P5.00mm_Vertical" (id 2) (at 65.405 192.659 0)
       (effects (font (size 1.27 1.27)) hide)
     )
@@
     )
     (path "/c2befb11-636d-44f8-aa20-c1ad551f3b77"
-      (reference "J6") (unit 1) (value "Conn_01x02") (footprint "")
+      (reference "J6") (unit 1) (value "Conn_01x02") (footprint "Connector_JST:JST_NV_B02P-NV_1x02_P5.00mm_Vertical")
     )
     (path "/00000000-0000-0000-0000-000061ef11ea/b1698c8b-d0cd-4216-a0b5-1b99da8a0202"
@@
     )
     (path "/00000000-0000-0000-0000-000061f130e5"
-      (reference "K1") (unit 1) (value "T9VV1K15-12S") (footprint "AERO-footprints:RELAY_T9VV1K15-12S")
+      (reference "K1") (unit 1) (value "T9VV1K15-12S") (footprint "AERO_Footprints:RELAY_T9VV1K15-12S")
     )
     (path "/00000000-0000-0000-0000-000062054c3a/00000000-0000-0000-0000-000062055384"
@@
       (reference "Q1") (unit 1) (value "B5584") (footprint "Package_TO_SOT_SMD:SOT-363_SC-70-6")
     )
+    (path "/00000000-0000-0000-0000-000061f4d99a/0051d338-4d08-4d10-938a-c63d3458c064"
+      (reference "Q2") (unit 1) (value "PSMN5R2-60YL") (footprint "Package_TO_SOT_SMD:LFPAK56")
+    )
     (path "/00000000-0000-0000-0000-000061f4d99a/51ade803-e43f-415b-acf1-cbe9b60e0555"
       (reference "Q3") (unit 1) (value "PSMN5R2-60YL") (footprint "Package_TO_SOT_SMD:LFPAK56")
@@
       (reference "Q4") (unit 1) (value "PSMN5R2-60YL") (footprint "Package_TO_SOT_SMD:LFPAK56")
     )
-    (path "/00000000-0000-0000-0000-000061f4d99a/0051d338-4d08-4d10-938a-c63d3458c064"
-      (reference "Q?") (unit 1) (value "PSMN5R2-60YL") (footprint "Package_TO_SOT_SMD:LFPAK56")
-    )
     (path "/9cd7a329-be98-4b6f-b451-5a50fe41a385"
       (reference "R2") (unit 1) (value "330") (footprint "Resistor_SMD:R_0603_1608Metric_Pad0.98x0.95mm_HandSolder")
@@
     )
     (path "/00000000-0000-0000-0000-000062054c3a/ec4b0bef-8187-4d99-b62c-b559b50cd5f8"
-      (reference "R10") (unit 1) (value "470") (footprint "")
+      (reference "R10") (unit 1) (value "470") (footprint "Resistor_SMD:R_0603_1608Metric_Pad0.98x0.95mm_HandSolder")
     )
     (path "/00000000-0000-0000-0000-000061f4d99a/78ff98dc-f3eb-4e0f-a212-b7188cae9868"
@@
     )
     (path "/00000000-0000-0000-0000-000061ef11ea/f9f1e0e1-c05e-4068-91f8-67895f3037cb"
-      (reference "U1") (unit 1) (value "Dev_Board_C") (footprint "")
+      (reference "U1") (unit 1) (value "Dev_Board_C") (footprint "esp32:ESP32-DevKitC")
     )
     (path "/dbb94e1e-e341-4f83-bcd9-f51be721f344"

Commit message: commit
Parts:
- added D10, D11, D12: FERD20M60ST, Package_TO_SOT_THT:TO-220-3_Vertical, symbol Simulation_SPICE:DIODE
Connections:
- net FuseBank/TSV is gone; now on net DCDC_IN: J1.23 (Pin_23)
- net BATT_12V: now also J1.7 (Pin_7), J1.8 (Pin_8); no longer J1.12 (Pin_12), J1.13 (Pin_13)
- net BRAKE_12V: now also D10.2 (K)
- net BRAKE_RTRN_12V: now also D10.1 (A)
- net BRB_RTN: now also J1.13 (Pin_13); no longer J1.20 (Pin_20)
- net DCDC_IN: now also J1.22 (Pin_22); no longer J1.7 (Pin_7), J1.8 (Pin_8)
- net FAN_12V: now also D11.2 (K)
- net FAN_RTRN_12V: now also D11.1 (A)
- net FAULT_BMS: now also J1.12 (Pin_12); no longer J1.22 (Pin_22)
- net PUMP_12V: now also D12.2 (K)
- net PUMP_RTRN_12V: now also D12.1 (A)
- net WATER_IN-: now also J2.8 (Pin_8); no longer J2.15 (Pin_15)
- net WATER_OUT-: now also J2.15 (Pin_15); no longer J2.8 (Pin_8)
- net BMS_12V: now reaches J2.12 (Pin_12)
- new net TSV: J1.20 (Pin_20)

Commit message: update
Connections:
- net FuseBank/BRB_LOOP is gone; now on net GND: J1.17 (Pin_17)
- net FuseBank/FRONT_12V is gone; now on net PUMP_RTRN_12V: J1.16 (Pin_16)
- net FuseBank/HVB_12 is gone; now on net FAN_RTRN_12V: J1.1 (Pin_1)
- net FuseBank/RINE_12V is gone; now on net PUMP_12V: J1.9 (Pin_9)
- net BATT_12V: now also J1.12 (Pin_12), J1.13 (Pin_13), J1.14 (Pin_14), J1.15 (Pin_15); no longer J1.5 (Pin_5), J1.6 (Pin_6), J1.7 (Pin_7), J1.8 (Pin_8)
- net BMS_12V: now also J1.6 (Pin_6); no longer J2.12 (Pin_12)
- net BRAKE_RTRN_12V: now also J1.3 (Pin_3); no longer J2.3 (Pin_3)
- net BRB_RTN: now also J3.8 (Pin_8); no longer J1.13 (Pin_13)
- net DCDC_IN: now also J1.20 (Pin_20), J1.21 (Pin_21); no longer J1.14 (Pin_14), J1.15 (Pin_15)
- net FAN_12V: now also J1.2 (Pin_2); no longer J1.3 (Pin_3)
- net FAN_RTRN_12V: no longer J2.4 (Pin_4)
- net FAULT_BMS: now also J1.7 (Pin_7); no longer J1.12 (Pin_12)
- net FAULT_IMD: now also J1.8 (Pin_8); no longer J1.21 (Pin_21)
- net GND: no longer J1.19 (Pin_19), J3.8 (Pin_8)
- net PUMP_12V: no longer J1.2 (Pin_2)
- net PUMP_RTRN_12V: no longer J2.5 (Pin_5)
- net TSV: now also J3.7 (Pin_7); no longer J1.20 (Pin_20)
- net BRB_LOOP: now reaches J3.1 (Pin_1)
- net RINE_12: now reaches J3.6 (Pin_6)
- new net FRONT_12: J1.19 (Pin_19)
- new net HVB_12: J1.5 (Pin_5)
Other:
- note removed: "For Shielding"

Commit message: DONE!!!!!
Connections:
- net SUSPENSION_L: now also J2.5 (Pin_5); no longer J2.14 (Pin_14)
- net SUSPENSION_R: now also J2.4 (Pin_4); no longer J2.7 (Pin_7)
- net WHEEL_L: now also J2.7 (Pin_7); no longer J2.13 (Pin_13)
Changed lines of the file:
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@@
+    (stroke (width 0) (type default) (color 0 0 0 0))
+  )
+  (wire (pts (xy 43.18 116.84) (xy 24.13 116.84))
     (stroke (width 0) (type default) (color 0 0 0 0))
   )
@@
     (stroke (width 0) (type default) (color 0 0 0 0))
   )
+  (wire (pts (xy 24.13 111.76) (xy 43.053 111.76))
+    (stroke (width 0) (type default) (color 0 0 0 0))
+  )
   (wire (pts (xy 147.574 188.468) (xy 155.829 188.468))
     (stroke (width 0) (type default) (color 0 0 0 0))
@@
     (stroke (width 0) (type default) (color 0 0 0 0))
   )
-  (wire (pts (xy 43.815 134.62) (xy 24.13 134.62))
-    (stroke (width 0) (type default) (color 0 0 0 0))
-  )
   (wire (pts (xy 89.535 57.15) (xy 89.535 59.69))
     (stroke (width 0) (type default) (color 0 0 0 0))
   )
+  (wire (pts (xy 43.053 109.22) (xy 24.13 109.22))
+    (stroke (width 0) (type default) (color 0 0 0 0))
+  )
   (wire (pts (xy 167.64 45.72) (xy 179.07 45.72))
     (stroke (width 0) (type default) (color 0 0 0 0))
@@
     (stroke (width 0) (type default) (color 0 0 0 0))
   )
-  (wire (pts (xy 43.18 116.84) (xy 24.13 116.84))
-    (stroke (width 0) (type default) (color 0 0 0 0))
-  )
   (wire (pts (xy 95.885 57.15) (xy 89.535 57.15))
     (stroke (width 0) (type default) (color 0 0 0 0))
@@
     (stroke (width 0) (type default) (color 0 0 0 0))
   )
-  (wire (pts (xy 43.815 132.08) (xy 24.13 132.08))
+  (wire (pts (xy 24.13 114.3) (xy 42.926 114.3))
     (stroke (width 0) (type default) (color 0 0 0 0))
   )
@@
   )
   (wire (pts (xy 24.13 139.7) (xy 44.45 139.7))
-    (stroke (width 0) (type default) (color 0 0 0 0))
-  )
-  (wire (pts (xy 43.815 114.3) (xy 24.13 114.3))
     (stroke (width 0) (type default) (color 0 0 0 0))
   )
@@
     (effects (font (size 1.27 1.27)) (justify left bottom))
   )
-  (label "SUSPENSION_L" (at 43.815 134.62 180)
+  (label "SUSPENSION_L" (at 43.053 111.76 180)
     (effects (font (size 1.27 1.27)) (justify right bottom))
   )
@@
     (effects (font (size 1.27 1.27)) (justify left bottom))
   )
-  (label "WHEEL_R" (at 43.815 114.3 180)
+  (label "WHEEL_R" (at 42.926 114.3 180)
     (effects (font (size 1.27 1.27)) (justify right bottom))
   )
@@
     (effects (font (size 1.27 1.27)) (justify left bottom))
   )
-  (label "WHEEL_L" (at 43.815 132.08 180)
+  (label "WHEEL_L" (at 43.18 116.84 180)
     (effects (font (size 1.27 1.27)) (justify right bottom))
   )
@@
     (effects (font (size 1.27 1.27)) (justify right bottom))
   )
-  (label "SUSPENSION_R" (at 43.18 116.84 180)
-    (effects (font (size 1.27 1.27)) (justify right bottom))
-  )
+  (label "SUSPENSION_R" (at 43.053 109.22 180)
+    (effects (font (size 1.27 1.27)) (justify right bottom))
+  )

Commit message: colin
Connections:
- net BATT_12V renamed Bat_12
Other:
- note added: "Should be SSOK here?"
Changed lines of the file:
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@@
     (stroke (width 0) (type default) (color 0 0 0 0))
   )
-  (wire (pts (xy 200.025 153.035) (xy 208.915 153.035))
+  (wire (pts (xy 200.152 153.035) (xy 208.915 153.035))
     (stroke (width 0) (type default) (color 0 0 0 0))
   )
@@
   )
   (text "Comes from HVB\nand BMS directly" (at 104.14 80.645 0)
+    (effects (font (size 1.27 1.27)) (justify left bottom))
+  )
+  (text "Should be SSOK here?" (at 187.833 156.972 0)
     (effects (font (size 1.27 1.27)) (justify left bottom))
   )
@@
     (effects (font (size 1.27 1.27)) (justify left bottom))
   )
-  (label "BRB_RTN" (at 200.025 153.035 0)
+  (label "BRB_RTN" (at 200.152 153.035 0)
     (effects (font (size 1.27 1.27)) (justify left bottom))
   )
@@
       (effects (font (size 1.27 1.27)) (justify right) hide)
     )
+  )
+  (global_label "Bat_12" (shape input) (at 89.535 54.61 180) (fields_autoplaced)
+    (effects (font (size 1.27 1.27)) (justify right))
+    (property "Intersheet References" "${INTERSHEET_REFS}" (id 0) (at 80.6794 54.5306 0)
+      (effects (font (size 1.27 1.27)) (justify right) hide)
+    )
