File: HVB High Voltage Board V1/high-voltage-board.kicad_pcb (KiCad board)
At the start: 2 copper layers, 179.2 x 115.7 mm, 43 parts, among them J1 Conn_01x23, J11 HV-, J2 Conn_01x02, J5 HV+, J6 HV-, J8 HV+, J9 Bender-LV, Q1 PSMN5R2-60YL, Q2 PSMN5R2-60YL, U2 LTV-817S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

Commit message: V1 with all Gerbers
Changed lines of the file:
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@@
       (drillshape 0)
       (scaleselection 1)
-      (outputdirectory "High_Voltage_Gerber/")
+      (outputdirectory "../BOARD GERBER/V1/HVB/")
     )
   )
@@
   (gr_arc (start 146.558 52.197) (mid 141.217488 50.41444) (end 139.065 45.212) (layer "Edge.Cuts") (width 0.1))
   (gr_arc (start 49.824325 152.435876) (mid 48.159536 151.687665) (end 47.411325 150.022876) (layer "Edge.Cuts") (width 0.1))
-  (gr_arc (start 136.3726 132.4864) (mid 134.25171 134.531549) (end 132.18101 132.4356) (layer "Edge.Cuts") (width 0.1))
+  (gr_arc (start 136.3726 132.4864) (mid 134.251711 134.531549) (end 132.18101 132.4356) (layer "Edge.Cuts") (width 0.1))
   (gr_line (start 161.788974 145.024974) (end 223.037528 145.059528) (layer "Edge.Cuts") (width 0.1))
   (gr_arc (start 137.9728 116.4844) (mid 137.786813 116.933413) (end 137.3378 117.1194) (layer "Edge.Cuts") (width 0.1))
