File: pacman/pacman.kicad_pcb (KiCad board)
At the start: 2 copper layers, 90.2 x 66 mm, 19 parts, among them J1 Conn_01x08, J3 Conn_01x01, J4 Conn_01x01, J5 Conn_01x01, J6 Conn_01x02, J9 JST PH, K1 G2RL, K2 G5V-1, K3 G5V-1, Q2 MMBT2222A

Commit message: V1 with all Gerbers
Changed lines of the file:
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@@
       (drillshape 0)
       (scaleselection 1)
-      (outputdirectory "Pac1_Gerber/")
+      (outputdirectory "../BOARD GERBER/V1/Pac1/")
     )
   )
@@
   (gr_line (start 201.422 49.53) (end 116.205 49.53) (layer "Edge.Cuts") (width 0.1))
   (gr_line (start 203.835 113.03) (end 203.835 52.07) (layer "Edge.Cuts") (width 0.1))
-  (gr_arc (start 201.422 49.53) (mid 203.130658 50.32087) (end 203.835 52.07) (layer "Edge.Cuts") (width 0.05))
+  (gr_arc (start 201.422 49.53) (mid 203.131697 50.321963) (end 203.835 52.07) (layer "Edge.Cuts") (width 0.05))
   (gr_arc (start 145.669 57.531) (mid 147.32 55.88) (end 148.971 57.531) (layer "Edge.Cuts") (width 0.1))
   (gr_line (start 148.971 61.595) (end 148.971 57.531) (layer "Edge.Cuts") (width 0.1))
