File: pacman_side_2/pacman_side_2.kicad_pcb (KiCad board)
At the start: 2 copper layers, 92.7 x 66.2 mm, 19 parts, among them J1 Conn_01x08, J3 Conn_01x01, J4 Conn_01x01, J5 Conn_01x01, J6 Conn_01x02, J9 JST PH, K1 G2RL, K2 G5V-1, K3 G5V-1, Q2 MMBT2222A

Commit message: Pac2 Cleanup
Parts:
- moved J3 1.05 mm to (177.1, 122.2)
- moved R1 0.38 mm to (179.3, 113.1)
Routing:
- net unconnected-(J1-Pad5): track 35.4 -> 0.00 mm
- net unconnected-(J1-Pad8): track 35.3 -> 0.00 mm
- net +12V: track 114.5 -> 92.3 mm
- net /INT+: track 24.4 -> 22.0 mm
- net Net-(D1-Pad2): track 19.2 -> 18.3 mm
